File: Hardware/RFSA3713-EVAL/RFSA3713-EVAL.kicad_sch (KiCad schematic)
At the start: 17 parts, among them J1 Conn_Coaxial, J2 Conn_Coaxial, J4 Conn_Coaxial, J5 Conn_Coaxial, J6 Conn_02x05_Odd_Even, SW1 SW_SPDT, SW2 SW_SPDT, SW3 SW_SPDT

Commit message: DRC and header re-sizing
Parts:
- J6: footprint Connector_PinHeader_1.00mm:PinHeader_2x05_P1.00mm_Vertical -> Connector_PinHeader_2.00mm:PinHeader_2x05_P2.00mm_Vertical
Changed lines of the file:
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@@
 			)
 		)
-		(property "Footprint" "Connector_PinHeader_1.00mm:PinHeader_2x05_P1.00mm_Vertical"
+		(property "Footprint" "Connector_PinHeader_2.00mm:PinHeader_2x05_P2.00mm_Vertical"
 			(at 208.28 86.36 0)
 			(effects
