File: Hardware/TX_Board/TX_Board.kicad_sch (KiCad schematic)
At the start: 48 parts, among them IC1 GP2Y1+, IC2 GP2Y1+, IC3 GP2Y1+, IC4 LT3041ADE#PBF, IC5 LT3099ADE#PBF, IC6 ADPL40502AUJZ-1.5-R7, J1 Conn_Coaxial, J10 MM8030-2610RJ3, J11 MM8030-2610RJ3, J12 MM8030-2610RJ3, J2 Conn_01x01_Pin, J25 Conn_02x14_Odd_Even, J3 Conn_01x01_Pin, J4 Conn_01x01_Pin, J5 Conn_01x01_Pin, J7 Conn_01x03_Socket, J8 Conn_02x08_Odd_Even, J9 MM8030-2610RJ3, U1 SN74HCT138NSR

Commit message: Final DRC review
Parts:
- J1: footprint Connector_Coaxial:SMA_Amphenol_132289_EdgeMount -> Connector_Coaxial:SMA_Samtec_SMA-J-P-H-ST-EM1_EdgeMount
Changed lines of the file:
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@@
 			)
 		)
-		(property "Footprint" "Connector_Coaxial:SMA_Amphenol_132289_EdgeMount"
+		(property "Footprint" "Connector_Coaxial:SMA_Samtec_SMA-J-P-H-ST-EM1_EdgeMount"
 			(at 29.21 116.84 0)
 			(effects
