File: Hardware/TX_Board/TX_Board.kicad_sch (KiCad schematic)
At the start: 48 parts, among them IC1 GP2Y1+, IC2 GP2Y1+, IC3 GP2Y1+, IC4 LT3041ADE#PBF, IC5 LT3099ADE#PBF, IC6 ADPL40502AUJZ-1.5-R7, J1 Conn_Coaxial, J10 MM8030-2610RJ3, J11 MM8030-2610RJ3, J12 MM8030-2610RJ3, J2 Conn_01x01_Pin, J3 Conn_01x01_Pin, J4 Conn_01x01_Pin, J5 Conn_01x01_Pin, J6 Conn_02x12_Odd_Even, J7 Conn_01x03_Socket, J8 Conn_02x08_Odd_Even, J9 MM8030-2610RJ3, U1 SN74HCT138NSR

Commit message: Ease of construction, added new layers, prelimininary routing.
Parts:
- C4, C5: footprint Capacitor_SMD:C_0402_1005Metric -> Capacitor_SMD:C_0603_1608Metric
- J2, J3, J4, J5: footprint Connector_PinHeader_2.00mm:PinHeader_1x01_P2.00mm_Vertical -> Connector_PinHeader_2.54mm:PinHeader_1x01_P2.54mm_Vertical
- J6: footprint Connector_PinHeader_2.00mm:PinHeader_2x12_P2.00mm_Vertical -> Connector_PinHeader_2.54mm:PinHeader_2x12_P2.54mm_Vertical
- J7: footprint Connector_PinSocket_2.00mm:PinSocket_1x03_P2.00mm_Vertical -> Connector_PinSocket_2.54mm:PinSocket_1x03_P2.54mm_Vertical
- J8: footprint Connector_PinHeader_2.00mm:PinHeader_2x08_P2.00mm_Vertical -> Connector_PinHeader_2.54mm:PinHeader_2x08_P2.54mm_Vertical
- R1, R10, R11, R2, R3, R5, R6, R7, R8, R9: footprint Resistor_SMD:R_0402_1005Metric -> Resistor_SMD:R_0603_1608Metric
Changed lines of the file:
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@@
 			)
 		)
-		(property "Footprint" "Connector_PinHeader_2.00mm:PinHeader_1x01_P2.00mm_Vertical"
+		(property "Footprint" "Connector_PinHeader_2.54mm:PinHeader_1x01_P2.54mm_Vertical"
 			(at 53.34 364.49 0)
 			(effects
@@
 			)
 		)
-		(property "Footprint" "Connector_PinSocket_2.00mm:PinSocket_1x03_P2.00mm_Vertical"
+		(property "Footprint" "Connector_PinSocket_2.54mm:PinSocket_1x03_P2.54mm_Vertical"
 			(at 73.66 345.44 0)
 			(effects
@@
 			)
 		)
-		(property "Footprint" "Resistor_SMD:R_0402_1005Metric"
+		(property "Footprint" "Resistor_SMD:R_0603_1608Metric"
 			(at 80.264 239.014 90)
 			(effects
@@
 			)
 		)
-		(property "Footprint" "Connector_PinHeader_2.00mm:PinHeader_1x01_P2.00mm_Vertical"
+		(property "Footprint" "Connector_PinHeader_2.54mm:PinHeader_1x01_P2.54mm_Vertical"
 			(at 53.34 359.41 0)
 			(effects
@@
 			)
 		)
-		(property "Footprint" "Resistor_SMD:R_0402_1005Metric"
+		(property "Footprint" "Resistor_SMD:R_0603_1608Metric"
 			(at 76.454 233.934 90)
 			(effects
@@
 			)
 		)
-		(property "Footprint" "Connector_PinHeader_2.00mm:PinHeader_2x08_P2.00mm_Vertical"
+		(property "Footprint" "Connector_PinHeader_2.54mm:PinHeader_2x08_P2.54mm_Vertical"
 			(at 121.92 269.24 0)
 			(effects
@@
 			)
 		)
-		(property "Footprint" "Connector_PinHeader_2.00mm:PinHeader_1x01_P2.00mm_Vertical"
+		(property "Footprint" "Connector_PinHeader_2.54mm:PinHeader_1x01_P2.54mm_Vertical"
 			(at 53.34 370.84 0)
 			(effects
@@
 			)
 		)
-		(property "Footprint" "Resistor_SMD:R_0402_1005Metric"
+		(property "Footprint" "Resistor_SMD:R_0603_1608Metric"
 			(at 76.454 231.394 90)
 			(effects
@@
 			)
 		)
-		(property "Footprint" "Resistor_SMD:R_0402_1005Metric"
+		(property "Footprint" "Resistor_SMD:R_0603_1608Metric"
 			(at 153.924 241.554 90)
 			(effects
@@
 			)
 		)
-		(property "Footprint" "Resistor_SMD:R_0402_1005Metric"
+		(property "Footprint" "Resistor_SMD:R_0603_1608Metric"
 			(at 153.924 231.394 90)
 			(effects
@@
 			)
 		)
-		(property "Footprint" "Resistor_SMD:R_0402_1005Metric"
+		(property "Footprint" "Resistor_SMD:R_0603_1608Metric"
 			(at 153.924 239.014 90)
 			(effects
@@
 			)
 		)
-		(property "Footprint" "Capacitor_SMD:C_0402_1005Metric"
+		(property "Footprint" "Capacitor_SMD:C_0603_1608Metric"
 			(at 166.0652 224.79 0)
 			(effects
@@
 			)
 		)
-		(property "Footprint" "Resistor_SMD:R_0402_1005Metric"
+		(property "Footprint" "Resistor_SMD:R_0603_1608Metric"
 			(at 153.924 226.314 90)
 			(effects
@@
 			)
 		)
-		(property "Footprint" "Resistor_SMD:R_0402_1005Metric"
+		(property "Footprint" "Resistor_SMD:R_0603_1608Metric"
 			(at 153.924 233.934 90)
 			(effects
@@
 			)
 		)
-		(property "Footprint" "Capacitor_SMD:C_0402_1005Metric"
+		(property "Footprint" "Capacitor_SMD:C_0603_1608Metric"
 			(at 157.1752 224.79 0)
 			(effects
@@
 			)
 		)
-		(property "Footprint" "Connector_PinHeader_2.00mm:PinHeader_1x01_P2.00mm_Vertical"
+		(property "Footprint" "Connector_PinHeader_2.54mm:PinHeader_1x01_P2.54mm_Vertical"
 			(at 53.34 375.92 0)
 			(effects
@@
 			)
 		)
-		(property "Footprint" "Resistor_SMD:R_0402_1005Metric"
+		(property "Footprint" "Resistor_SMD:R_0603_1608Metric"
 			(at 153.924 228.854 90)
 			(effects
@@
 			)
 		)
-		(property "Footprint" "Connector_PinHeader_2.00mm:PinHeader_2x12_P2.00mm_Vertical"
+		(property "Footprint" "Connector_PinHeader_2.54mm:PinHeader_2x12_P2.54mm_Vertical"
 			(at 58.42 297.18 0)
 			(effects
@@
 			)
 		)
-		(property "Footprint" "Resistor_SMD:R_0402_1005Metric"
+		(property "Footprint" "Resistor_SMD:R_0603_1608Metric"
 			(at 153.924 236.474 90)
 			(effects

Commit message: more routing
Connections:
- net ATTN_LE_1: now also J8.7 (Pin_7), J8.8 (Pin_8), R8.2; no longer J8.3 (Pin_3), J8.4 (Pin_4), R6.2
- net ATTN_LE_2: now also J8.5 (Pin_5), J8.6 (Pin_6), R7.2; no longer J8.7 (Pin_7), J8.8 (Pin_8), R8.2
- net ATTN_LE_3: now also J8.3 (Pin_3), J8.4 (Pin_4), R6.2; no longer J8.11 (Pin_11), J8.12 (Pin_12), R10.2
- net ATTN_LE_4: now also J8.1 (Pin_1), J8.2 (Pin_2), R5.2; no longer J8.15 (Pin_15), J8.16 (Pin_16), R3.1
- net PS_LE_1: now also J8.15 (Pin_15), J8.16 (Pin_16), R3.1; no longer J8.1 (Pin_1), J8.2 (Pin_2), R5.2
- net PS_LE_2: now also J8.13 (Pin_13), J8.14 (Pin_14), R11.2; no longer J8.5 (Pin_5), J8.6 (Pin_6), R7.2
- net PS_LE_3: now also J8.11 (Pin_11), J8.12 (Pin_12), R10.2; no longer J8.10 (Pin_10), J8.9 (Pin_9), R9.2
- net PS_LE_4: now also J8.10 (Pin_10), J8.9 (Pin_9), R9.2; no longer J8.13 (Pin_13), J8.14 (Pin_14), R11.2

Commit message: DRC and more layout
Connections:
- net ATTN_A0: no longer J6.19 (Pin_19), J6.20 (Pin_20)
- net ATTN_A1: no longer J6.21 (Pin_21), J6.22 (Pin_22)
- net ATTN_A2: no longer J6.23 (Pin_23), J6.24 (Pin_24)
- net GND: now also J6.19 (Pin_19), J6.20 (Pin_20), J6.21 (Pin_21), J6.22 (Pin_22), J6.23 (Pin_23), J6.24 (Pin_24)

Commit message: Gerbers
Parts:
- R4: footprint Resistor_SMD:R_0201_0603Metric -> Resistor_SMD:R_0603_1608Metric
Changed lines of the file:
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@@
 			)
 		)
-		(property "Footprint" "Resistor_SMD:R_0201_0603Metric"
+		(property "Footprint" "Resistor_SMD:R_0603_1608Metric"
 			(at 122.174 346.964 90)
 			(effects

Commit message: Testing Data
Parts:
- removed J6: Conn_02x12_Odd_Even, Connector_PinHeader_2.54mm:PinHeader_2x12_P2.54mm_Vertical, symbol tx_board_symbol_library:Conn_02x12_Odd_Even
- added J25: Conn_02x14_Odd_Even, Connector_PinHeader_2.54mm:PinHeader_2x14_P2.54mm_Horizontal, symbol Connector_Generic:Conn_02x14_Odd_Even
- J1: footprint Connector_Coaxial:SMA_Amphenol_132289_EdgeMount -> Connector_Coaxial:SMA_Samtec_SMA-J-P-H-ST-EM1_EdgeMount
- J8: footprint Connector_PinHeader_2.54mm:PinHeader_2x08_P2.54mm_Vertical -> Connector_PinHeader_2.54mm:PinHeader_2x08_P2.54mm_Horizontal
- R12, R13, R14, R15, R16, R17: footprint Resistor_SMD:R_0201_0603Metric -> Resistor_SMD:R_0603_1608Metric
Connections:
- net ATTN_CLK: now also J25.17 (Pin_17), J25.18 (Pin_18)
- net ATTN_SI: now also J25.15 (Pin_15), J25.16 (Pin_16)
- net GND: now also J25.19 (Pin_19), J25.20 (Pin_20)
- net GPIO0: now also J25.1 (Pin_1), J25.2 (Pin_2)
- net GPIO1: now also J25.3 (Pin_3), J25.4 (Pin_4)
- net GPIO2: now also J25.5 (Pin_5), J25.6 (Pin_6)
- net GPIO3: now also J25.7 (Pin_7), J25.8 (Pin_8)
- net PS_CLK: now also J25.11 (Pin_11), J25.12 (Pin_12)
- net PS_SER_IN: now also J25.10 (Pin_10), J25.9 (Pin_9)
- net PS_SER_OUT: now also J25.13 (Pin_13), J25.14 (Pin_14)
- net VCC: now also J25.21 (Pin_21), J25.22 (Pin_22)
- net VEE: now also J25.23 (Pin_23), J25.24 (Pin_24)
- net V_PD: now also J25.25 (Pin_25), J25.26 (Pin_26)
- no-connect marks 7 -> 9

Commit message: Begin Rev 2
Parts:
- added S1: SLW-865144-2A-N-SMT-TR, SLW-865144-2A-N-SMT-TR:SW_SLW-865144-2A-N-SMT-TR, symbol SLW-865144-2A-N-SMT-TR:SLW-865144-2A-N-SMT-TR
Connections:
- net GND: now also S1.1
- net VCC: now also S1.3; no longer IC6.3 (EN)
- new net: IC6.3 (EN), S1.2
