File: Hardware/ADP5071_Power_Supply/KiCad/ADP5071_Dual_Supply.kicad_pcb (KiCad board)
At the start: 2 copper layers, 59.4 x 36.9 mm, 43 parts, among them J1 MountingPin, J2 Screw_Terminal_01x02, J3 Conn_01x03_Pin, J4 MountingPin, J5 MountingPin, J6 MountingPin, U1 ADP5071AREZ

Commit message: Testing Data
Parts:
- added J7: Conn_01x03_Pin, Connector_PinHeader_2.54mm:PinHeader_1x03_P2.54mm_Horizontal, F.Cu at (107.5, 81.3)
Routing:
- net Net-(U1-VREG): track 95.4 -> 99.4 mm
- net +VDC: track 41.4 -> 45.0 mm
- net -VDC: track 43.9 -> 47.1 mm
- net GNDREF: vias 41 -> 45
