File: Hardware/ADP5071_Power_Supply/KiCad/ADP5071_Dual_Supply.kicad_sch (KiCad schematic)
At the start: 42 parts, among them J1 MountingPin, J2 Screw_Terminal_01x02, J3 Conn_01x03_Pin, J4 MountingPin, J5 MountingPin, J6 MountingPin, U1 ADP5071AREZ

Commit message: Ease of construction, added new layers, prelimininary routing.
Parts:
- J1, J4, J5, J6: footprint Connector_PinSocket_2.00mm:PinSocket_1x01_P2.00mm_Vertical -> Connector_PinSocket_2.54mm:PinSocket_1x01_P2.54mm_Vertical
- J3: footprint Connector_PinHeader_2.00mm:PinHeader_1x03_P2.00mm_Vertical -> Connector_PinHeader_2.54mm:PinHeader_1x03_P2.54mm_Vertical
Changed lines of the file:
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@@
 			)
 		)
-		(property "Footprint" "Connector_PinHeader_2.00mm:PinHeader_1x03_P2.00mm_Vertical"
+		(property "Footprint" "Connector_PinHeader_2.54mm:PinHeader_1x03_P2.54mm_Vertical"
 			(at 213.36 82.55 0)
 			(effects
@@
 			)
 		)
-		(property "Footprint" "Connector_PinSocket_2.00mm:PinSocket_1x01_P2.00mm_Vertical"
+		(property "Footprint" "Connector_PinSocket_2.54mm:PinSocket_1x01_P2.54mm_Vertical"
 			(at 223.52 158.75 0)
 			(effects
@@
 			)
 		)
-		(property "Footprint" "Connector_PinSocket_2.00mm:PinSocket_1x01_P2.00mm_Vertical"
+		(property "Footprint" "Connector_PinSocket_2.54mm:PinSocket_1x01_P2.54mm_Vertical"
 			(at 223.52 152.4 0)
 			(effects
@@
 			)
 		)
-		(property "Footprint" "Connector_PinSocket_2.00mm:PinSocket_1x01_P2.00mm_Vertical"
+		(property "Footprint" "Connector_PinSocket_2.54mm:PinSocket_1x01_P2.54mm_Vertical"
 			(at 240.03 158.75 0)
 			(effects
@@
 			)
 		)
-		(property "Footprint" "Connector_PinSocket_2.00mm:PinSocket_1x01_P2.00mm_Vertical"
+		(property "Footprint" "Connector_PinSocket_2.54mm:PinSocket_1x01_P2.54mm_Vertical"
 			(at 240.03 152.4 0)
 			(effects

Commit message: Testing Data
Parts:
- added J7: Conn_01x03_Pin, Connector_PinHeader_2.54mm:PinHeader_1x03_P2.54mm_Horizontal, symbol Connector:Conn_01x03_Pin
Connections:
- net +VDC: now also J7.1 (Pin_1)
- net -VDC: now also J7.3 (Pin_3)
- net GNDREF: now also J7.2 (Pin_2)
Changed lines of the file:
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@@
 	(text "-V Out"
 		(exclude_from_sim no)
-		(at 222.25 85.852 0)
+		(at 221.742 67.818 0)
 		(effects
 			(font
@@
 	(text "GND"
 		(exclude_from_sim no)
-		(at 220.218 83.566 0)
+		(at 220.472 70.612 0)
 		(effects
 			(font
@@
 		)
 	)
+	(text "GND"
+		(exclude_from_sim no)
+		(at 218.44 83.566 0)
+		(effects
+			(font
+				(size 1.27 1.27)
+			)
+			(justify right bottom)
+		)
+	)
 	(text "+V Out"
 		(exclude_from_sim no)
-		(at 221.996 81.026 0)
+		(at 220.98 81.026 0)
+		(effects
+			(font
+				(size 1.27 1.27)
+			)
+			(justify right bottom)
+		)
+	)
+	(text "+V Out"
+		(exclude_from_sim no)
+		(at 222.25 73.152 0)
 		(effects
 			(font
@@
 		)
 	)
+	(text "-V Out"
+		(exclude_from_sim no)
+		(at 221.234 86.106 0)
+		(effects
+			(font
+				(size 1.27 1.27)
+			)
+			(justify right bottom)
+		)
+	)
 	(junction
 		(at 160.02 100.33)
@@
 	)
 	(junction
+		(at 205.74 85.09)
+		(diameter 0)
+		(color 0 0 0 0)
+	)
+	(junction
 		(at 190.5 80.01)
 		(diameter 0)
@@
 	)
 	(junction
+		(at 200.66 80.01)
+		(diameter 0)
+		(color 0 0 0 0)
+	)
+	(junction
 		(at 60.96 85.09)
 		(diameter 0)
@@
 	)
 	(junction
+		(at 203.2 82.55)
+		(diameter 0)
+		(color 0 0 0 0)
+	)
+	(junction
 		(at 80.01 85.09)
 		(diameter 0)
@@
 	(wire
 		(pts
+			(xy 203.2 69.85) (xy 203.2 82.55)
+		)
+		(stroke
+			(width 0)
+			(type default)
+		)
+	)
+	(wire
+		(pts
 			(xy 162.56 105.41) (xy 172.72 105.41)
 		)
@@
 	(wire
 		(pts
-			(xy 190.5 80.01) (xy 208.28 80.01)
+			(xy 190.5 80.01) (xy 200.66 80.01)
 		)
 		(stroke
@@
 	(wire
 		(pts
+			(xy 200.66 72.39) (xy 200.66 80.01)
+		)
+		(stroke
+			(width 0)
+			(type default)
+		)
+	)
+	(wire
+		(pts
 			(xy 76.2 76.2) (xy 80.01 76.2)
 		)
@@
 	(wire
 		(pts
+			(xy 208.28 69.85) (xy 203.2 69.85)
+		)
+		(stroke
+			(width 0)
+			(type default)
+		)
+	)
+	(wire
+		(pts
 			(xy 92.71 104.14) (xy 92.71 111.76)
 		)
@@
 	(wire
 		(pts
+			(xy 208.28 67.31) (xy 205.74 67.31)
+		)
+		(stroke
+			(width 0)
+			(type default)
+		)
+	)
+	(wire
+		(pts
+			(xy 200.66 80.01) (xy 208.28 80.01)
+		)
+		(stroke
+			(width 0)
+			(type default)
+		)
+	)
+	(wire
+		(pts
 			(xy 128.27 82.55) (xy 127 82.55)
 		)
@@
 	(wire
 		(pts
-			(xy 190.5 102.87) (xy 207.01 102.87)
+			(xy 190.5 102.87) (xy 205.74 102.87)
 		)
 		(stroke
@@
 	(wire
 		(pts
+			(xy 205.74 67.31) (xy 205.74 85.09)
+		)
+		(stroke
+			(width 0)
+			(type default)
+		)
+	)
+	(wire
+		(pts
 			(xy 127 110.49) (xy 127 120.65)
 		)
@@
 	(wire
 		(pts
-			(xy 207.01 102.87) (xy 207.01 85.09)
+			(xy 205.74 102.87) (xy 205.74 85.09)
 		)
 		(stroke
@@
 	(wire
 		(pts
+			(xy 200.66 72.39) (xy 208.28 72.39)
+		)
+		(stroke
+			(width 0)
+			(type default)
+		)
+	)
+	(wire
+		(pts
 			(xy 67.31 69.85) (xy 69.85 69.85)
 		)
@@
 	(wire
 		(pts
-			(xy 207.01 85.09) (xy 208.28 85.09)
+			(xy 205.74 85.09) (xy 208.28 85.09)
 		)
 		(stroke
@@
 					(unit 1)
 				)
+			)
+		)
+	)
+	(symbol
+		(lib_id "Connector:Conn_01x03_Pin")
+		(at 213.36 69.85 180)
+		(unit 1)
+		(exclude_from_sim no)
+		(in_bom yes)
+		(on_board yes)
+		(dnp no)
+		(fields_autoplaced yes)
+		(property "Reference" "J7"
+			(at 214.63 68.5799 0)
+			(effects
+				(font
+					(size 1.27 1.27)
+				)
+				(justify right)
+			)
+		)
+		(property "Value" "Conn_01x03_Pin"
+			(at 214.63 71.1199 0)
+			(effects
+				(font
+					(size 1.27 1.27)
+				)
+				(justify right)
+			)
+		)
+		(property "Footprint" "Connector_PinHeader_2.54mm:PinHeader_1x03_P2.54mm_Horizontal"
+			(at 213.36 69.85 0)
+			(effects
+				(font
+					(size 1.27 1.27)
+				)
+				(hide yes)
+			)
+		)
+		(property "Datasheet" "~"
+			(at 213.36 69.85 0)
+			(effects
+				(font
+					(size 1.27 1.27)
+				)
+				(hide yes)
+			)
+		)
+		(property "Description" "Generic connector, single row, 01x03, script generated"
+			(at 213.36 69.85 0)
+			(effects
+				(font
+					(size 1.27 1.27)
+				)
+				(hide yes)
+			)
+		)
+		(pin "3"
+		)
+		(pin "1"
+		)
+		(pin "2"
+		)
+		(instances
+			(project ""
+				(path "/359c8d50-ab92-45cb-a3ea-95ee484a708c"
+					(reference "J7")
+					(unit 1)
+				)
