File: Hardware/TX_Board_Rev2/TX_Board_Rev2.kicad_pcb (KiCad board)
At the start: 2 copper layers, 104.6 x 87.3 mm, 293 parts, among them IC1 GP2Y1+, IC10 PE42423B-Z, IC11 MAPS-010164-TR0500, IC12 PE42423B-Z, IC13 QPA9122TR7, IC14 PMA3-63GLN+, IC15 PMA3-63GLN+, IC16 PE42423B-Z, IC17 MAPS-010164-TR0500, IC18 PE42423B-Z, IC19 PE42423B-Z, IC2 GP2Y1+, IC20 QPA9122TR7, IC21 PMA3-63GLN+, IC22 PE42423B-Z, IC23 PE42423B-Z, IC24 ADP5600ACPZ-R7, IC25 TPS7A4701RGWT, IC27 ADPL40502AUJZ-1.8-R7, IC3 GP2Y1+, IC4 MAPS-010164-TR0500, IC5 QPA9122TR7, IC6 MAPS-010164-TR0500, IC7 PE42423B-Z, IC8 QPA9122TR7, IC9 PMA3-63GLN+, J1 Conn_Coaxial, J10 MM8030-2610RJ3, J11 MM8030-2610RJ3, J12 MM8030-2610RJ3, J13 Conn_Coaxial, J14 Conn_Coaxial, J15 MM8030-2610RJ3, J16 Conn_Coaxial, J17 Conn_Coaxial, J19 694106301002, J2 MM8030-2610RJ3, J20 Conn_01x08, J3 MM8030-2610RJ3, J4 Conn_Coaxial, J5 Conn_Coaxial, J6 Conn_Coaxial, J7 Conn_Coaxial, J8 MM8030-2610RJ3, J9 MM8030-2610RJ3, U1 SN74HCT138NSR

Commit message: Rev 2 progress
Parts:
- C134: footprint Capacitor_SMD:C_0603_1608Metric -> Capacitor_SMD:C_0402_1005Metric
- JP1, JP2: footprint Connector_PinHeader_2.54mm:PinHeader_1x11_P2.54mm_Vertical -> Connector_PinSocket_2.54mm:PinSocket_1x11_P2.54mm_Vertical
- moved C139 102.0 mm to (159.2, 61.2), turned to 90 degrees
- moved C142 100.4 mm to (151.0, 59.8), turned to 90 degrees
- moved C140 96.9 mm to (153.7, 65.3), turned to 180 degrees
- moved C144 96.0 mm to (168.8, 63.8), turned to 90 degrees
- moved C145 95.7 mm to (163.8, 61.4), turned to -90 degrees
- moved C143 95.3 mm to (167.2, 60.5)
- moved IC27 89.4 mm to (166.3, 63.4), turned to -90 degrees
- moved C135 87.8 mm to (142.4, 57.0)
- moved IC25 86.4 mm to (155.1, 61.2), turned to 180 degrees
- moved C133 84.9 mm to (140.2, 58.5)
- moved C137 82.9 mm to (138.1, 62.5), turned to 90 degrees
- moved R59 81.6 mm to (141.2, 64.7)
- moved C138 80.5 mm to (150.5, 62.2)
- moved C136 76.1 mm to (145.2, 60.8), turned to 90 degrees
- moved R7 75.7 mm to (117.8, 61.2)
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Connections:
- J20 pad 1: ATTN_LE_4 -> ATTN_LE_3
- J20 pad 2: ATTN_LE_3 -> ATTN_LE_2
- J20 pad 3: ATTN_LE_2 -> ATTN_LE_1
- J20 pad 4: ATTN_LE_1 -> ATTN_LE_0
- J20 pad 5: PS_LE_4 -> PS_LE_3
- J20 pad 6: PS_LE_3 -> PS_LE_2
- J20 pad 7: PS_LE_2 -> PS_LE_1
- J20 pad 8: PS_LE_1 -> PS_LE_0
- JP1 pad 3: unconnected-(JP1-Pad3) -> GND
- R10 pad 2: PS_LE_3 -> PS_LE_2
- R11 pad 2: PS_LE_2 -> PS_LE_1
- R20 pad 2: /Channel1/PS_LE_0 -> PS_LE_1
- R24 pad 2: /Channel1/ATTN_LE_0 -> ATTN_LE_1
- R3 pad 1: PS_LE_1 -> PS_LE_0
- R31 pad 2: /Channel2/PS_LE_0 -> PS_LE_2
- R37 pad 2: /Channel2/ATTN_LE_0 -> ATTN_LE_2
- R43 pad 2: /Channel3/PS_LE_0 -> PS_LE_3
- R47 pad 2: /Channel3/ATTN_LE_0 -> ATTN_LE_3
- R5 pad 2: ATTN_LE_4 -> ATTN_LE_3
- R6 pad 2: ATTN_LE_3 -> ATTN_LE_2
- R7 pad 2: ATTN_LE_2 -> ATTN_LE_1
- R8 pad 2: ATTN_LE_1 -> ATTN_LE_0
- R9 pad 2: PS_LE_4 -> PS_LE_3
Routing:
- net VEE: track 2.91 -> 74.8 mm, vias 0 -> 6
- net V_PD: track 3.90 -> 71.9 mm, vias 0 -> 5
- net VCC: track 33.0 -> 76.1 mm, vias 0 -> 39
- net SER_IN: track 0.00 -> 7.86 mm, vias 0 -> 8
- net GPIO3: track 0.00 -> 7.78 mm
- net CLK: track 0.00 -> 7.56 mm, vias 0 -> 8
- net GPIO2: track 0.00 -> 7.25 mm
- net GPIO1: track 0.00 -> 6.72 mm
- net Net-(IC24-CPOUT_1): track 0.00 -> 5.71 mm
- net Net-(IC24-C1-): track 0.00 -> 2.12 mm
- net ATTN_LE_3: track 0.00 -> 1.97 mm, vias 0 -> 2
- net ATTN_LE_2: track 0.00 -> 1.97 mm, vias 0 -> 2
- net ATTN_LE_1: track 0.00 -> 1.97 mm, vias 0 -> 2
- net ATTN_LE_0: track 0.00 -> 1.97 mm, vias 0 -> 2
- net V_EN: track 0.00 -> 1.97 mm
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- added copper zone on In1.Cu, net GND
- added copper zone on In2.Cu, net VCC
- added copper zone on F.Cu, net VDC
- added copper zone on F.Cu, net VEE
Other:
- copper layers 2 -> 4
- board text added: "GND"
- board text added: "VCC"
- board text added: "VDC"
- board text added: "VEE"
