File: Hardware/TX_Board_Rev2/channel1.kicad_sch (KiCad schematic)
At the start: 65 parts, among them IC10 PE42423B-Z, IC6 MAPS-010164-TR0500, IC7 PE42423B-Z, IC8 QPA9122TR7, IC9 PMA3-63GLN+, J2 MM8030-2610RJ3, J6 Conn_Coaxial, J7 Conn_Coaxial

Commit message: Rev2 layout partially complete
Parts:
- removed R28: 51, Resistor_SMD:R_0603_1608Metric, symbol tx_board_symbol_library:R_US
- removed R34: 50, Resistor_SMD:R_0402_1005Metric, symbol tx_board_symbol_library:R_US
- AT1: footprint tx_board_footprints:QFN50P300X300X90-17N -> RFSA3713:QFN50P300X300X90-17N
- C13, C14, C15, C16, C17, C18, C19, C20, C21, C22, C23, C24, C25, C26, C27, C32, C33, C34, C52, C53, C54, C58, C59: footprint Capacitor_SMD:C_0603_1608Metric -> Capacitor_SMD:C_0402_1005Metric
- C28, C29, C56, C57: value C_Small -> 22 pF; footprint (none) -> Capacitor_SMD:C_0402_1005Metric
- C31, C55: footprint Capacitor_SMD:C_0402_1005Metric_Pad0.74x0.62mm_HandSolder -> Capacitor_SMD:C_0402_1005Metric
- C35: footprint Capacitor_SMD:C_0603_1608Metric_Pad1.08x0.95mm_HandSolder -> Capacitor_SMD:C_0402_1005Metric
- C51: footprint Capacitor_SMD:C_1206_3216Metric_Pad1.33x1.80mm_HandSolder -> Capacitor_SMD:C_0402_1005Metric
- IC10, IC7: footprint PE42423B-Z:QFN50P300X300X90-17N-D -> PE42423:QFN50P300X300X90-17N-D
- IC6: footprint tx_board_footprints:QFN50P400X400X100-25N-D -> MAPS-010164-TR0500:QFN50P400X400X100-25N-D
- IC8: footprint tx_board_footprints:QPA9122TR7 -> QPA9122-TR7:QPA9122TR7
- J2: footprint tx_board_footprints:MM80302610RJ3 -> MM8030-2610RJ3:MM80302610RJ3
- R18, R19, R20, R21, R22, R23, R24, R25: footprint Resistor_SMD:R_0603_1608Metric -> Resistor_SMD:R_0402_1005Metric
- R26: value 0 -> 51; footprint Resistor_SMD:R_0603_1608Metric -> Resistor_SMD:R_0402_1005Metric
- R27: value 0 -> 50; footprint Resistor_SMD:R_0603_1608Metric -> Resistor_SMD:R_0402_1005Metric
Connections:
- net GND: now also R27.2
- net VCC: now also C53.2, C54.1, R26.1; no longer R27.2
- net V_PD: now also C32.2, L15.1; no longer R26.1
- net at IC8.13 (VBIAS): now also R26.2
- net at HY1.5 (COUPLED_(REVERSE)): now also R27.1
- net ATTN_LE_1 renamed ATTN_LE_0
- net PS_LE_1 renamed PS_LE_0

Commit message: Rev 2 progress
Connections:
- net ATTN_LE_0 renamed ATTN_LE_1
- net PS_LE_0 renamed PS_LE_1
Changed lines of the file:
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@@
 		)
 	)
-	(hierarchical_label "PS_LE_0"
+	(hierarchical_label "PS_LE_1"
 		(shape input)
 		(at 276.86 226.06 0)
@@
 		)
 	)
-	(hierarchical_label "ATTN_LE_0"
+	(hierarchical_label "ATTN_LE_1"
 		(shape input)
 		(at 386.08 267.97 0)

Commit message: Rev2 Complete
Parts:
- removed J6: Conn_Coaxial, Connector_Coaxial:SMA_Samtec_SMA-J-P-H-ST-EM1_EdgeMount, symbol Connector:Conn_Coaxial
- added J4: CONSMA022-G, CONSMA022_G:LINX_CONSMA022-G, symbol CONSMA022-G:CONSMA022-G
- added R53, R54: 20k, Resistor_SMD:R_0402_1005Metric, symbol Device:R_US
Connections:
- net GND: now also J4.2, J4.3, J4.4, J4.5, R53.2; no longer IC7.15 (LS)
- net OUTPUT: now also J4.1
- net VCC: now also R54.1; no longer IC10.15 (LS)
- new net: IC10.15 (LS), R54.2
- new net: IC7.15 (LS), R53.1
