File: Hardware/TX_Board_Rev2/channel2.kicad_sch (KiCad schematic)
At the start: 65 parts, among them IC11 MAPS-010164-TR0500, IC12 PE42423B-Z, IC13 QPA9122TR7, IC14 PMA3-63GLN+, IC16 PE42423B-Z, J13 MM8030-2610RJ3, J14 Conn_Coaxial, J15 Conn_Coaxial

Commit message: Rev2 layout partially complete
Parts:
- removed J13: MM8030-2610RJ3, tx_board_footprints:MM80302610RJ3, symbol tx_board_symbol_library:MM8030-2610RJ3
- removed J15: Conn_Coaxial, Connector_Coaxial:SMA_Amphenol_901-144_Vertical, symbol Connector:Conn_Coaxial
- removed R41: 50, Resistor_SMD:R_0603_1608Metric, symbol tx_board_symbol_library:R_US
- removed R42: 8.2, Resistor_SMD:R_0603_1608Metric, symbol tx_board_symbol_library:R_US
- removed R43, R44: 0, Resistor_SMD:R_0603_1608Metric, symbol tx_board_symbol_library:R_US
- removed R45: 51, Resistor_SMD:R_0603_1608Metric, symbol tx_board_symbol_library:R_US
- removed R46: 50, Resistor_SMD:R_0402_1005Metric, symbol tx_board_symbol_library:R_US
- added J13: Conn_Coaxial, Connector_Coaxial:SMA_Samtec_SMA-J-P-H-ST-EM1_EdgeMount, symbol Connector:Conn_Coaxial
- added J8: MM8030-2610RJ3, MM8030-2610RJ3:MM80302610RJ3, symbol tx_board_symbol_library:MM8030-2610RJ3
- added R28, R30, R31, R34: 50, Resistor_SMD:R_0402_1005Metric, symbol tx_board_symbol_library:R_US
- AT3: footprint tx_board_footprints:QFN50P300X300X90-17N -> RFSA3713:QFN50P300X300X90-17N
- C61, C62, C63, C64, C65, C66, C67, C68, C69, C70, C71, C72, C73, C74, C75, C80, C81, C82, C85, C86, C87, C91, C92: footprint Capacitor_SMD:C_0603_1608Metric -> Capacitor_SMD:C_0402_1005Metric
- C76, C77, C89, C90: value C_Small -> 22 pF; footprint (none) -> Capacitor_SMD:C_0402_1005Metric
- C79, C88: footprint Capacitor_SMD:C_0402_1005Metric_Pad0.74x0.62mm_HandSolder -> Capacitor_SMD:C_0402_1005Metric
- C83: footprint Capacitor_SMD:C_0603_1608Metric_Pad1.08x0.95mm_HandSolder -> Capacitor_SMD:C_0402_1005Metric
- C84: footprint Capacitor_SMD:C_1206_3216Metric_Pad1.33x1.80mm_HandSolder -> Capacitor_SMD:C_0402_1005Metric
- IC11: footprint tx_board_footprints:QFN50P400X400X100-25N-D -> MAPS-010164-TR0500:QFN50P400X400X100-25N-D
- IC12, IC16: footprint PE42423B-Z:QFN50P300X300X90-17N-D -> PE42423:QFN50P300X300X90-17N-D
- IC13: footprint tx_board_footprints:QPA9122TR7 -> QPA9122-TR7:QPA9122TR7
- J14: footprint Connector_Coaxial:SMA_Samtec_SMA-J-P-H-ST-EM1_EdgeMount -> Connector_Coaxial:SMA_Amphenol_901-144_Vertical
- R35, R36, R37, R40: footprint Resistor_SMD:R_0603_1608Metric -> Resistor_SMD:R_0402_1005Metric
- R38: value 50 -> 8.2; footprint Resistor_SMD:R_0603_1608Metric -> Resistor_SMD:R_0402_1005Metric
- R39: value 50 -> 51; footprint Resistor_SMD:R_0603_1608Metric -> Resistor_SMD:R_0402_1005Metric
Connections:
- net ATTN-RF_OUT: now also J8.1 (IN)
- net CLK: now also R36.2, R30.1; no longer R36.1, R40.2
- net CPL_FWD: now also J14.1 (In)
- net GND: now also R40.2, J13.2 (Ext), J8.3 (GND_1), J8.4 (GND_2)
- net OUTPUT: now also J13.1 (In); no longer J14.1 (In)
- net SER_IN: now also R28.1; no longer R39.1
- net SER_OUT: now also R34.1; no longer R38.1
- net VCC: now also C86.2, C87.1, R39.1
- net V_PD: now also C80.2, L25.1
- net at IC13.13 (VBIAS): now also R39.2
- net at C81.1, L24.2: now also R38.1
- net at AT3.12 (LE), C75.2: now also R37.1
- net at C67.2, IC11.22 (D3_OR_LE): now also R31.1; no longer R37.1
- net at AT3.13 (CLK), C74.1: now also R36.1; no longer R40.1
- net at HY3.5 (COUPLED_(REVERSE)): now also R40.1
- net at C66.2, IC11.23 (D2_OR_CLK): now also R30.2; no longer R36.2
- net at C65.1, IC11.24 (D1_OR_SER_IN): now also R28.2; no longer R35.2
- net at IC13.4 (VCC1/VCC2): now also R38.2
- net at AT3.14 (SI), C73.1: now also R35.2; no longer R39.2
- net at IC12.7 (RFC): now also J8.2 (OUT)
- net at C70.1, IC11.17 (SER_OUT): now also R34.2; no longer R38.2
- net PS_LE_2 renamed ATTN_LE_0
- new net PS_LE_0: R31.2

Commit message: Rev 2 progress
Connections:
- net ATTN_LE_0 renamed ATTN_LE_2
- net PS_LE_0 renamed PS_LE_2
Changed lines of the file:
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@@
 		)
 	)
-	(hierarchical_label "ATTN_LE_0"
+	(hierarchical_label "ATTN_LE_2"
 		(shape input)
 		(at 405.13 280.67 0)
@@
 		)
 	)
-	(hierarchical_label "PS_LE_0"
+	(hierarchical_label "PS_LE_2"
 		(shape input)
 		(at 295.91 238.76 0)

Commit message: Rev2 Complete
Parts:
- removed J13: Conn_Coaxial, Connector_Coaxial:SMA_Samtec_SMA-J-P-H-ST-EM1_EdgeMount, symbol Connector:Conn_Coaxial
- added J6: CONSMA022-G, CONSMA022_G:LINX_CONSMA022-G, symbol CONSMA022-G:CONSMA022-G
- added R55, R56: 20k, Resistor_SMD:R_0402_1005Metric, symbol Device:R_US
Connections:
- net GND: now also J6.2, J6.3, J6.4, J6.5, R55.2; no longer IC12.15 (LS)
- net OUTPUT: now also J6.1
- net VCC: now also R56.1; no longer IC16.15 (LS)
- new net: IC16.15 (LS), R56.2
- new net: IC12.15 (LS), R55.1

Commit message: Rev 3, rotated interface connectors
Parts:
- renumbered AT3 to AT2, HY3 to CPL2, J14 to CPL_PORT2, J8 to J10, J6 to J2, IC14 to LNA2, IC13 to PA2, IC11 to PS2, IC12 to SW20, IC16 to SW21
Changed lines of the file:
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@@
 		(on_board yes)
 		(dnp no)
-		(property "Reference" "IC14"
+		(property "Reference" "LNA2"
 			(at 550.672 326.136 0)
 			(effects
@@
 			(project "TX_Board_Rev2"
 				(path "/5327d041-dca0-47c6-802d-ce81714adf6c/f15f633c-4a68-465c-891b-a0907b206a37"
-					(reference "IC14")
+					(reference "LNA2")
 					(unit 1)
 				)
@@
 		(dnp no)
 		(fields_autoplaced yes)
-		(property "Reference" "HY3"
+		(property "Reference" "CPL2"
 			(at 689.61 266.7 0)
 			(effects
@@
 			(project "TX_Board_Rev2"
 				(path "/5327d041-dca0-47c6-802d-ce81714adf6c/f15f633c-4a68-465c-891b-a0907b206a37"
-					(reference "HY3")
+					(reference "CPL2")
 					(unit 1)
 				)
@@
 		(dnp no)
 		(fields_autoplaced yes)
-		(property "Reference" "J14"
+		(property "Reference" "CPL_PORT2"
 			(at 739.14 264.4531 0)
 			(effects
@@
 			(project "TX_Board_Rev2"
 				(path "/5327d041-dca0-47c6-802d-ce81714adf6c/f15f633c-4a68-465c-891b-a0907b206a37"
-					(reference "J14")
+					(reference "CPL_PORT2")
 					(unit 1)
 				)
@@
 		(dnp no)
 		(fields_autoplaced yes)
-		(property "Reference" "IC16"
+		(property "Reference" "SW21"
 			(at 606.4819 289.56 90)
 			(effects
@@
 			(project "TX_Board_Rev2"
 				(path "/5327d041-dca0-47c6-802d-ce81714adf6c/f15f633c-4a68-465c-891b-a0907b206a37"
-					(reference "IC16")
+					(reference "SW21")
 					(unit 1)
 				)
@@
 		(dnp no)
 		(fields_autoplaced yes)
-		(property "Reference" "AT3"
+		(property "Reference" "AT2"
 			(at 382.27 274.2498 0)
 			(effects
@@
 			(project "TX_Board_Rev2"
 				(path "/5327d041-dca0-47c6-802d-ce81714adf6c/f15f633c-4a68-465c-891b-a0907b206a37"
-					(reference "AT3")
+					(reference "AT2")
 					(unit 1)
 				)
@@
 		(on_board yes)
 		(dnp no)
-		(property "Reference" "IC11"
+		(property "Reference" "PS2"
 			(at 298.45 271.7098 0)
 			(effects
@@
 			(project "TX_Board_Rev2"
 				(path "/5327d041-dca0-47c6-802d-ce81714adf6c/f15f633c-4a68-465c-891b-a0907b206a37"
-					(reference "IC11")
+					(reference "PS2")
 					(unit 1)
 				)
@@
 		(dnp no)
 		(fields_autoplaced yes)
-		(property "Reference" "IC13"
+		(property "Reference" "PA2"
 			(at 570.23 232.3398 0)
 			(effects
@@
 			(project "TX_Board_Rev2"
 				(path "/5327d041-dca0-47c6-802d-ce81714adf6c/f15f633c-4a68-465c-891b-a0907b206a37"
-					(reference "IC13")
+					(reference "PA2")
 					(unit 1)
 				)
@@
 		(dnp no)
 		(fields_autoplaced yes)
-		(property "Reference" "J6"
+		(property "Reference" "J2"
 			(at 721.5505 285.75 0)
 			(effects
@@
 			(project "TX_Board_Rev2"
 				(path "/5327d041-dca0-47c6-802d-ce81714adf6c/f15f633c-4a68-465c-891b-a0907b206a37"
-					(reference "J6")
+					(reference "J2")
 					(unit 1)
 				)
@@
 		(on_board yes)
 		(dnp no)
-		(property "Reference" "J8"
+		(property "Reference" "J10"
 			(at 430.022 309.626 90)
 			(effects
@@
 			(project "TX_Board_Rev2"
 				(path "/5327d041-dca0-47c6-802d-ce81714adf6c/f15f633c-4a68-465c-891b-a0907b206a37"
-					(reference "J8")
+					(reference "J10")
 					(unit 1)
 				)
@@
 		(dnp no)
 		(fields_autoplaced yes)
-		(property "Reference" "IC12"
+		(property "Reference" "SW20"
 			(at 475.5581 273.05 90)
 			(effects
@@
 			(project "TX_Board_Rev2"
 				(path "/5327d041-dca0-47c6-802d-ce81714adf6c/f15f633c-4a68-465c-891b-a0907b206a37"
-					(reference "IC12")
+					(reference "SW20")
 					(unit 1)
 				)

Commit message: Restored broken Rev 2 for posterity and cleaned up naming
Parts:
- renumbered AT2 to AT3, CPL2 to HY3, PS2 to IC11, SW20 to IC12, PA2 to IC13, LNA2 to IC14, SW21 to IC16, CPL_PORT2 to J14, J2 to J6, J10 to J8
Changed lines of the file:
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@@
 		(on_board yes)
 		(dnp no)
-		(property "Reference" "LNA2"
+		(property "Reference" "IC14"
 			(at 550.672 326.136 0)
 			(effects
@@
 			(project "TX_Board_Rev2"
 				(path "/5327d041-dca0-47c6-802d-ce81714adf6c/f15f633c-4a68-465c-891b-a0907b206a37"
-					(reference "LNA2")
+					(reference "IC14")
 					(unit 1)
 				)
@@
 		(dnp no)
 		(fields_autoplaced yes)
-		(property "Reference" "CPL2"
+		(property "Reference" "HY3"
 			(at 689.61 266.7 0)
 			(effects
@@
 			(project "TX_Board_Rev2"
 				(path "/5327d041-dca0-47c6-802d-ce81714adf6c/f15f633c-4a68-465c-891b-a0907b206a37"
-					(reference "CPL2")
+					(reference "HY3")
 					(unit 1)
 				)
@@
 		(dnp no)
 		(fields_autoplaced yes)
-		(property "Reference" "CPL_PORT2"
+		(property "Reference" "J14"
 			(at 739.14 264.4531 0)
 			(effects
@@
 			(project "TX_Board_Rev2"
 				(path "/5327d041-dca0-47c6-802d-ce81714adf6c/f15f633c-4a68-465c-891b-a0907b206a37"
-					(reference "CPL_PORT2")
+					(reference "J14")
 					(unit 1)
 				)
@@
 		(dnp no)
 		(fields_autoplaced yes)
-		(property "Reference" "SW21"
+		(property "Reference" "IC16"
 			(at 606.4819 289.56 90)
 			(effects
@@
 			(project "TX_Board_Rev2"
 				(path "/5327d041-dca0-47c6-802d-ce81714adf6c/f15f633c-4a68-465c-891b-a0907b206a37"
-					(reference "SW21")
+					(reference "IC16")
 					(unit 1)
 				)
@@
 		(dnp no)
 		(fields_autoplaced yes)
-		(property "Reference" "AT2"
+		(property "Reference" "AT3"
 			(at 382.27 274.2498 0)
 			(effects
@@
 			(project "TX_Board_Rev2"
 				(path "/5327d041-dca0-47c6-802d-ce81714adf6c/f15f633c-4a68-465c-891b-a0907b206a37"
-					(reference "AT2")
+					(reference "AT3")
 					(unit 1)
 				)
@@
 		(on_board yes)
 		(dnp no)
-		(property "Reference" "PS2"
+		(property "Reference" "IC11"
 			(at 298.45 271.7098 0)
 			(effects
@@
 			(project "TX_Board_Rev2"
 				(path "/5327d041-dca0-47c6-802d-ce81714adf6c/f15f633c-4a68-465c-891b-a0907b206a37"
-					(reference "PS2")
+					(reference "IC11")
 					(unit 1)
 				)
@@
 		(dnp no)
 		(fields_autoplaced yes)
-		(property "Reference" "PA2"
+		(property "Reference" "IC13"
 			(at 570.23 232.3398 0)
 			(effects
@@
 			(project "TX_Board_Rev2"
 				(path "/5327d041-dca0-47c6-802d-ce81714adf6c/f15f633c-4a68-465c-891b-a0907b206a37"
-					(reference "PA2")
+					(reference "IC13")
 					(unit 1)
 				)
@@
 		(dnp no)
 		(fields_autoplaced yes)
-		(property "Reference" "J2"
+		(property "Reference" "J6"
 			(at 721.5505 285.75 0)
 			(effects
@@
 			(project "TX_Board_Rev2"
 				(path "/5327d041-dca0-47c6-802d-ce81714adf6c/f15f633c-4a68-465c-891b-a0907b206a37"
-					(reference "J2")
+					(reference "J6")
 					(unit 1)
 				)
@@
 		(on_board yes)
 		(dnp no)
-		(property "Reference" "J10"
+		(property "Reference" "J8"
 			(at 430.022 309.626 90)
 			(effects
@@
 			(project "TX_Board_Rev2"
 				(path "/5327d041-dca0-47c6-802d-ce81714adf6c/f15f633c-4a68-465c-891b-a0907b206a37"
-					(reference "J10")
+					(reference "J8")
 					(unit 1)
 				)
@@
 		(dnp no)
 		(fields_autoplaced yes)
-		(property "Reference" "SW20"
+		(property "Reference" "IC12"
 			(at 475.5581 273.05 90)
 			(effects
@@
 			(project "TX_Board_Rev2"
 				(path "/5327d041-dca0-47c6-802d-ce81714adf6c/f15f633c-4a68-465c-891b-a0907b206a37"
-					(reference "SW20")
+					(reference "IC12")
 					(unit 1)
 				)
