File: Hardware/TX_Board_Rev2/channel3.kicad_sch (KiCad schematic)
At the start: 65 parts, among them IC17 MAPS-010164-TR0500, IC18 PE42423B-Z, IC20 QPA9122TR7, IC21 PMA3-63GLN+, IC22 PE42423B-Z, J16 MM8030-2610RJ3, J17 Conn_Coaxial, J18 Conn_Coaxial

Commit message: Rev2 layout partially complete
Parts:
- removed J16: MM8030-2610RJ3, tx_board_footprints:MM80302610RJ3, symbol tx_board_symbol_library:MM8030-2610RJ3
- removed J18: Conn_Coaxial, Connector_Coaxial:SMA_Amphenol_901-144_Vertical, symbol Connector:Conn_Coaxial
- removed R51, R52, R53: 50, Resistor_SMD:R_0603_1608Metric, symbol tx_board_symbol_library:R_US
- removed R54: 8.2, Resistor_SMD:R_0603_1608Metric, symbol tx_board_symbol_library:R_US
- removed R55, R56: 0, Resistor_SMD:R_0603_1608Metric, symbol tx_board_symbol_library:R_US
- removed R57: 51, Resistor_SMD:R_0603_1608Metric, symbol tx_board_symbol_library:R_US
- removed R58: 50, Resistor_SMD:R_0402_1005Metric, symbol tx_board_symbol_library:R_US
- added J15: MM8030-2610RJ3, MM8030-2610RJ3:MM80302610RJ3, symbol tx_board_symbol_library:MM8030-2610RJ3
- added J16: Conn_Coaxial, Connector_Coaxial:SMA_Samtec_SMA-J-P-H-ST-EM1_EdgeMount, symbol Connector:Conn_Coaxial
- added R41, R42, R43, R44, R45, R46: 50, Resistor_SMD:R_0402_1005Metric, symbol tx_board_symbol_library:R_US
- AT4: footprint tx_board_footprints:QFN50P300X300X90-17N -> RFSA3713:QFN50P300X300X90-17N
- C100, C101, C102, C103, C104, C105, C106, C107, C108, C117, C118, C119, C122, C123, C124, C128, C131, C94, C95, C96, C97, C98, C99: footprint Capacitor_SMD:C_0603_1608Metric -> Capacitor_SMD:C_0402_1005Metric
- C109, C110, C126, C127: value C_Small -> 22 pF; footprint (none) -> Capacitor_SMD:C_0402_1005Metric
- C112, C125: footprint Capacitor_SMD:C_0402_1005Metric_Pad0.74x0.62mm_HandSolder -> Capacitor_SMD:C_0402_1005Metric
- C120: footprint Capacitor_SMD:C_0603_1608Metric_Pad1.08x0.95mm_HandSolder -> Capacitor_SMD:C_0402_1005Metric
- C121: footprint Capacitor_SMD:C_1206_3216Metric_Pad1.33x1.80mm_HandSolder -> Capacitor_SMD:C_0402_1005Metric
- IC17: footprint tx_board_footprints:QFN50P400X400X100-25N-D -> MAPS-010164-TR0500:QFN50P400X400X100-25N-D
- IC18, IC22: footprint PE42423B-Z:QFN50P300X300X90-17N-D -> PE42423:QFN50P300X300X90-17N-D
- IC20: footprint tx_board_footprints:QPA9122TR7 -> QPA9122-TR7:QPA9122TR7
- J17: footprint Connector_Coaxial:SMA_Samtec_SMA-J-P-H-ST-EM1_EdgeMount -> Connector_Coaxial:SMA_Amphenol_901-144_Vertical
- R47, R50: footprint Resistor_SMD:R_0603_1608Metric -> Resistor_SMD:R_0402_1005Metric
- R48: value 50 -> 8.2; footprint Resistor_SMD:R_0603_1608Metric -> Resistor_SMD:R_0402_1005Metric
- R49: value 50 -> 51; footprint Resistor_SMD:R_0603_1608Metric -> Resistor_SMD:R_0402_1005Metric
Connections:
- net PS_LE_3 is gone; now on an unnamed net: R49.2
- net ATTN-RF_OUT: now also J15.1 (IN)
- net CLK: now also R42.1, R46.2; no longer R48.1
- net CPL_FWD: now also J17.1 (In)
- net GND: now also R50.2, J15.3 (GND_1), J15.4 (GND_2), J16.2 (Ext)
- net OUTPUT: now also J16.1 (In); no longer J17.1 (In)
- net SER_IN: now also R41.1, R45.1; no longer R47.1
- net SER_OUT: now also R44.1; no longer R50.1
- net VCC: now also C123.2, C124.1, R49.1
- net V_PD: now also C117.2, L36.1
- net at C118.1, L35.2: now also R48.1
- net at AT4.12 (LE), C108.2: now also R47.1
- net at C100.2, IC17.22 (D3_OR_LE): now also R43.1; no longer R49.1
- net at AT4.13 (CLK), C107.1: now also R46.1
- net at HY4.5 (COUPLED_(REVERSE)): now also R50.1
- net at C99.2, IC17.23 (D2_OR_CLK): now also R42.2; no longer R48.2
- net at C98.1, IC17.24 (D1_OR_SER_IN): now also R41.2; no longer R47.2
- net at IC20.4 (VCC1/VCC2): now also R48.2
- net at AT4.14 (SI), C106.1: now also R45.2
- net at IC18.7 (RFC): now also J15.2 (OUT)
- net at C103.1, IC17.17 (SER_OUT): now also R44.2; no longer R50.2
- new net ATTN_LE_0: R47.2
- new net PS_LE_0: R43.2

Commit message: Rev 2 progress
Connections:
- net ATTN_LE_0 renamed ATTN_LE_3
- net PS_LE_0 renamed PS_LE_3
Changed lines of the file:
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@@
 		)
 	)
-	(hierarchical_label "PS_LE_0"
+	(hierarchical_label "PS_LE_3"
 		(shape input)
 		(at 260.35 255.27 0)
@@
 		)
 	)
-	(hierarchical_label "ATTN_LE_0"
+	(hierarchical_label "ATTN_LE_3"
 		(shape input)
 		(at 369.57 297.18 0)

Commit message: Rev2 Complete
Parts:
- removed J16: Conn_Coaxial, Connector_Coaxial:SMA_Samtec_SMA-J-P-H-ST-EM1_EdgeMount, symbol Connector:Conn_Coaxial
- added J13: CONSMA022-G, CONSMA022_G:LINX_CONSMA022-G, symbol CONSMA022-G:CONSMA022-G
- added R57, R58: 20k, Resistor_SMD:R_0402_1005Metric, symbol Device:R_US
Connections:
- net GND: now also J13.2, J13.3, J13.4, J13.5, R57.2; no longer IC18.15 (LS)
- net OUTPUT: now also J13.1
- net VCC: now also R58.1; no longer IC22.15 (LS)
- new net: IC18.15 (LS), R57.1
- new net: IC22.15 (LS), R58.2

Commit message: Rev 3, rotated interface connectors
Parts:
- renumbered AT4 to AT3, HY4 to CPL3, J17 to CPL_PORT3, J15 to J11, J13 to J3, IC21 to LNA3, IC20 to PA3, IC17 to PS3, IC18 to SW30, IC22 to SW31
Changed lines of the file:
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@@
 		(dnp no)
 		(fields_autoplaced yes)
-		(property "Reference" "IC20"
+		(property "Reference" "PA3"
 			(at 534.67 248.8498 0)
 			(effects
@@
 			(project "TX_Board_Rev2"
 				(path "/5327d041-dca0-47c6-802d-ce81714adf6c/f2c46e2d-52f6-42ae-b733-37434a659606"
-					(reference "IC20")
+					(reference "PA3")
 					(unit 1)
 				)
@@
 		(dnp no)
 		(fields_autoplaced yes)
-		(property "Reference" "IC18"
+		(property "Reference" "SW30"
 			(at 439.9981 289.56 90)
 			(effects
@@
 			(project "TX_Board_Rev2"
 				(path "/5327d041-dca0-47c6-802d-ce81714adf6c/f2c46e2d-52f6-42ae-b733-37434a659606"
-					(reference "IC18")
+					(reference "SW30")
 					(unit 1)
 				)
@@
 		(dnp no)
 		(fields_autoplaced yes)
-		(property "Reference" "HY4"
+		(property "Reference" "CPL3"
 			(at 654.05 283.21 0)
 			(effects
@@
 			(project "TX_Board_Rev2"
 				(path "/5327d041-dca0-47c6-802d-ce81714adf6c/f2c46e2d-52f6-42ae-b733-37434a659606"
-					(reference "HY4")
+					(reference "CPL3")
 					(unit 1)
 				)
@@
 		(on_board yes)
 		(dnp no)
-		(property "Reference" "J15"
+		(property "Reference" "J11"
 			(at 394.462 326.136 90)
 			(effects
@@
 			(project "TX_Board_Rev2"
 				(path "/5327d041-dca0-47c6-802d-ce81714adf6c/f2c46e2d-52f6-42ae-b733-37434a659606"
-					(reference "J15")
+					(reference "J11")
 					(unit 1)
 				)
@@
 		(dnp no)
 		(fields_autoplaced yes)
-		(property "Reference" "J17"
+		(property "Reference" "CPL_PORT3"
 			(at 703.58 280.9631 0)
 			(effects
@@
 			(project "TX_Board_Rev2"
 				(path "/5327d041-dca0-47c6-802d-ce81714adf6c/f2c46e2d-52f6-42ae-b733-37434a659606"
-					(reference "J17")
+					(reference "CPL_PORT3")
 					(unit 1)
 				)
@@
 		(on_board yes)
 		(dnp no)
-		(property "Reference" "IC21"
+		(property "Reference" "LNA3"
 			(at 515.112 342.646 0)
 			(effects
@@
 			(project "TX_Board_Rev2"
 				(path "/5327d041-dca0-47c6-802d-ce81714adf6c/f2c46e2d-52f6-42ae-b733-37434a659606"
-					(reference "IC21")
+					(reference "LNA3")
 					(unit 1)
 				)
@@
 		(dnp no)
 		(fields_autoplaced yes)
-		(property "Reference" "J13"
+		(property "Reference" "J3"
 			(at 685.9905 302.26 0)
 			(effects
@@
 			(project "TX_Board_Rev2"
 				(path "/5327d041-dca0-47c6-802d-ce81714adf6c/f2c46e2d-52f6-42ae-b733-37434a659606"
-					(reference "J13")
+					(reference "J3")
 					(unit 1)
 				)
@@
 		(on_board yes)
 		(dnp no)
-		(property "Reference" "IC17"
+		(property "Reference" "PS3"
 			(at 262.89 288.2198 0)
 			(effects
@@
 			(project "TX_Board_Rev2"
 				(path "/5327d041-dca0-47c6-802d-ce81714adf6c/f2c46e2d-52f6-42ae-b733-37434a659606"
-					(reference "IC17")
+					(reference "PS3")
 					(unit 1)
 				)
@@
 		(dnp no)
 		(fields_autoplaced yes)
-		(property "Reference" "AT4"
+		(property "Reference" "AT3"
 			(at 346.71 290.7598 0)
 			(effects
@@
 			(project "TX_Board_Rev2"
 				(path "/5327d041-dca0-47c6-802d-ce81714adf6c/f2c46e2d-52f6-42ae-b733-37434a659606"
-					(reference "AT4")
+					(reference "AT3")
 					(unit 1)
 				)
@@
 		(dnp no)
 		(fields_autoplaced yes)
-		(property "Reference" "IC22"
+		(property "Reference" "SW31"
 			(at 570.9219 306.07 90)
 			(effects
@@
 			(project "TX_Board_Rev2"
 				(path "/5327d041-dca0-47c6-802d-ce81714adf6c/f2c46e2d-52f6-42ae-b733-37434a659606"
-					(reference "IC22")
+					(reference "SW31")
 					(unit 1)
 				)

Commit message: Restored broken Rev 2 for posterity and cleaned up naming
Parts:
- renumbered AT3 to AT4, CPL3 to HY4, PS3 to IC17, SW30 to IC18, PA3 to IC20, LNA3 to IC21, SW31 to IC22, J3 to J13, J11 to J15, CPL_PORT3 to J17
Changed lines of the file:
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@@
 		(dnp no)
 		(fields_autoplaced yes)
-		(property "Reference" "PA3"
+		(property "Reference" "IC20"
 			(at 534.67 248.8498 0)
 			(effects
@@
 			(project "TX_Board_Rev2"
 				(path "/5327d041-dca0-47c6-802d-ce81714adf6c/f2c46e2d-52f6-42ae-b733-37434a659606"
-					(reference "PA3")
+					(reference "IC20")
 					(unit 1)
 				)
@@
 		(dnp no)
 		(fields_autoplaced yes)
-		(property "Reference" "SW30"
+		(property "Reference" "IC18"
 			(at 439.9981 289.56 90)
 			(effects
@@
 			(project "TX_Board_Rev2"
 				(path "/5327d041-dca0-47c6-802d-ce81714adf6c/f2c46e2d-52f6-42ae-b733-37434a659606"
-					(reference "SW30")
+					(reference "IC18")
 					(unit 1)
 				)
@@
 		(dnp no)
 		(fields_autoplaced yes)
-		(property "Reference" "CPL3"
+		(property "Reference" "HY4"
 			(at 654.05 283.21 0)
 			(effects
@@
 			(project "TX_Board_Rev2"
 				(path "/5327d041-dca0-47c6-802d-ce81714adf6c/f2c46e2d-52f6-42ae-b733-37434a659606"
-					(reference "CPL3")
+					(reference "HY4")
 					(unit 1)
 				)
@@
 		(on_board yes)
 		(dnp no)
-		(property "Reference" "J11"
+		(property "Reference" "J15"
 			(at 394.462 326.136 90)
 			(effects
@@
 			(project "TX_Board_Rev2"
 				(path "/5327d041-dca0-47c6-802d-ce81714adf6c/f2c46e2d-52f6-42ae-b733-37434a659606"
-					(reference "J11")
+					(reference "J15")
 					(unit 1)
 				)
@@
 		(dnp no)
 		(fields_autoplaced yes)
-		(property "Reference" "CPL_PORT3"
+		(property "Reference" "J17"
 			(at 703.58 280.9631 0)
 			(effects
@@
 			(project "TX_Board_Rev2"
 				(path "/5327d041-dca0-47c6-802d-ce81714adf6c/f2c46e2d-52f6-42ae-b733-37434a659606"
-					(reference "CPL_PORT3")
+					(reference "J17")
 					(unit 1)
 				)
@@
 		(on_board yes)
 		(dnp no)
-		(property "Reference" "LNA3"
+		(property "Reference" "IC21"
 			(at 515.112 342.646 0)
 			(effects
@@
 			(project "TX_Board_Rev2"
 				(path "/5327d041-dca0-47c6-802d-ce81714adf6c/f2c46e2d-52f6-42ae-b733-37434a659606"
-					(reference "LNA3")
+					(reference "IC21")
 					(unit 1)
 				)
@@
 		(dnp no)
 		(fields_autoplaced yes)
-		(property "Reference" "J3"
+		(property "Reference" "J13"
 			(at 685.9905 302.26 0)
 			(effects
@@
 			(project "TX_Board_Rev2"
 				(path "/5327d041-dca0-47c6-802d-ce81714adf6c/f2c46e2d-52f6-42ae-b733-37434a659606"
-					(reference "J3")
+					(reference "J13")
 					(unit 1)
 				)
@@
 		(on_board yes)
 		(dnp no)
-		(property "Reference" "PS3"
+		(property "Reference" "IC17"
 			(at 262.89 288.2198 0)
 			(effects
@@
 			(project "TX_Board_Rev2"
 				(path "/5327d041-dca0-47c6-802d-ce81714adf6c/f2c46e2d-52f6-42ae-b733-37434a659606"
-					(reference "PS3")
+					(reference "IC17")
 					(unit 1)
 				)
@@
 		(dnp no)
 		(fields_autoplaced yes)
-		(property "Reference" "AT3"
+		(property "Reference" "AT4"
 			(at 346.71 290.7598 0)
 			(effects
@@
 			(project "TX_Board_Rev2"
 				(path "/5327d041-dca0-47c6-802d-ce81714adf6c/f2c46e2d-52f6-42ae-b733-37434a659606"
-					(reference "AT3")
+					(reference "AT4")
 					(unit 1)
 				)
@@
 		(dnp no)
 		(fields_autoplaced yes)
-		(property "Reference" "SW31"
+		(property "Reference" "IC22"
 			(at 570.9219 306.07 90)
 			(effects
@@
 			(project "TX_Board_Rev2"
 				(path "/5327d041-dca0-47c6-802d-ce81714adf6c/f2c46e2d-52f6-42ae-b733-37434a659606"
-					(reference "SW31")
+					(reference "IC22")
 					(unit 1)
 				)
