File: Hardware/OpenPhasedArray0.3/channel0.kicad_sch (KiCad schematic)
At the start: 65 parts, among them IC10 PE42423B-Z, IC6 MAPS-010164-TR0500, IC7 PE42423B-Z, IC8 QPA9122TR7, IC9 PMA3-63GLN+, J2 MM8030-2610RJ3, J4 CONSMA022-G, J7 Conn_Coaxial

Commit message: Restored broken Rev 2 for posterity and cleaned up naming
Parts:
- removed AT1: RFSA3713TR7, RFSA3713:QFN50P300X300X90-17N, symbol tx_board_symbol_library:RFSA3713TR7
- removed C13, C14, C20: 0.1uF, Capacitor_SMD:C_0402_1005Metric, symbol tx_board_symbol_library:C
- removed C15, C16, C21: 100pF, Capacitor_SMD:C_0402_1005Metric, symbol tx_board_symbol_library:C
- removed C17, C18, C19, C22, C25, C26, C27: 1.3 pF, Capacitor_SMD:C_0402_1005Metric, symbol tx_board_symbol_library:C
- removed C23: 470p, Capacitor_SMD:C_0402_1005Metric, symbol tx_board_symbol_library:C
- removed C24: 1uF, Capacitor_SMD:C_0402_1005Metric, symbol tx_board_symbol_library:C
- removed C28, C29, C56, C57: 22 pF, Capacitor_SMD:C_0402_1005Metric, symbol Device:C_Small
- removed C30, C60: 18 pF, Capacitor_SMD:C_0402_1005Metric, symbol tx_board_symbol_library:C
- removed C31, C55: 18pF, Capacitor_SMD:C_0402_1005Metric, symbol Device:C
- removed C32, C34, C58: 1 uF, Capacitor_SMD:C_0402_1005Metric, symbol tx_board_symbol_library:C
- removed C33, C52, C53, C54, C59: 100 pF, Capacitor_SMD:C_0402_1005Metric, symbol tx_board_symbol_library:C
- removed C35: 100pF, Capacitor_SMD:C_0402_1005Metric, symbol Device:C
- removed C51: 10uF, Capacitor_SMD:C_0402_1005Metric, symbol Device:C
- removed HY1: BDCA1-10-40+, BDCA1-10-40+:BDCA11040, symbol BDCA1-10-40+:BDCA1-10-40+
- removed IC10, IC7: PE42423B-Z, PE42423:QFN50P300X300X90-17N-D, symbol PE42423B-Z:PE42423B-Z
- removed IC6: MAPS-010164-TR0500, MAPS-010164-TR0500:QFN50P400X400X100-25N-D, symbol tx_board_symbol_library:MAPS-010164-TR0500
- removed IC8: QPA9122TR7, QPA9122-TR7:QPA9122TR7, symbol tx_board_symbol_library:QPA9122TR7
- removed IC9: PMA3-63GLN+, PMA3-63GLN+:QFN51P300X300X89-13N, symbol PMA3-63GLN+:PMA3-63GLN+
- removed J2: MM8030-2610RJ3, MM8030-2610RJ3:MM80302610RJ3, symbol tx_board_symbol_library:MM8030-2610RJ3
- removed J4: CONSMA022-G, CONSMA022_G:LINX_CONSMA022-G, symbol CONSMA022-G:CONSMA022-G
- removed J7: Conn_Coaxial, Connector_Coaxial:SMA_Amphenol_901-144_Vertical, symbol Connector:Conn_Coaxial
- removed L12, L13, L14, L15, L17, L18, L5, L9: L_Ferrite, Inductor_SMD:L_0201_0603Metric_Pad0.64x0.40mm_HandSolder, symbol Device:L_Ferrite
- removed L16: 12nH, Inductor_SMD:L_0603_1608Metric_Pad1.05x0.95mm_HandSolder, symbol Device:L
- removed L19: 12 nH, Inductor_SMD:L_0603_1608Metric, symbol tx_board_symbol_library:L
- removed R18, R19, R20, R21, R22, R23, R24, R27: 50, Resistor_SMD:R_0402_1005Metric, symbol tx_board_symbol_library:R_US
- removed R25: 8.2, Resistor_SMD:R_0402_1005Metric, symbol tx_board_symbol_library:R_US
- removed R26: 51, Resistor_SMD:R_0402_1005Metric, symbol tx_board_symbol_library:R_US
- removed R53, R54: 20k, Resistor_SMD:R_0402_1005Metric, symbol Device:R_US
- added AT0: RFSA3713TR7, RFSA3713:QFN50P300X300X90-17N, symbol tx_board_symbol_library:RFSA3713TR7
- added C1, C10, C2: 0.1uF, Capacitor_SMD:C_0402_1005Metric, symbol tx_board_symbol_library:C
- added C11, C3, C6: 100pF, Capacitor_SMD:C_0402_1005Metric, symbol tx_board_symbol_library:C
- added C113, C116: 18pF, Capacitor_SMD:C_0402_1005Metric, symbol Device:C
- added C114: 10uF, Capacitor_SMD:C_0402_1005Metric, symbol Device:C
- added C115: 100pF, Capacitor_SMD:C_0402_1005Metric, symbol Device:C
- added C12, C38, C39, C40, C7, C8, C9: 1.3 pF, Capacitor_SMD:C_0402_1005Metric, symbol tx_board_symbol_library:C
- added C129, C130, C141, C149: 22 pF, Capacitor_SMD:C_0402_1005Metric, symbol Device:C_Small
- added C36: 470p, Capacitor_SMD:C_0402_1005Metric, symbol tx_board_symbol_library:C
- added C37: 1uF, Capacitor_SMD:C_0402_1005Metric, symbol tx_board_symbol_library:C
- added C41, C50: 18 pF, Capacitor_SMD:C_0402_1005Metric, symbol tx_board_symbol_library:C
- added C42, C44, C48: 1 uF, Capacitor_SMD:C_0402_1005Metric, symbol tx_board_symbol_library:C
- added C43, C45, C46, C47, C49: 100 pF, Capacitor_SMD:C_0402_1005Metric, symbol tx_board_symbol_library:C
- added CPL0: BDCA1-10-40+, BDCA1-10-40+:BDCA11040, symbol BDCA1-10-40+:BDCA1-10-40+
- added CPL_PORT0: Conn_Coaxial, Connector_Coaxial:SMA_Amphenol_901-144_Vertical, symbol Connector:Conn_Coaxial
- added J0: CONSMA022-G, CONSMA022_G:LINX_CONSMA022-G, symbol CONSMA022-G:CONSMA022-G
- added J8: MM8030-2610RJ3, MM8030-2610RJ3:MM80302610RJ3, symbol tx_board_symbol_library:MM8030-2610RJ3
- added L1, L10, L2, L3, L4, L6, L7, L8: L_Ferrite, Inductor_SMD:L_0201_0603Metric_Pad0.64x0.40mm_HandSolder, symbol Device:L_Ferrite
- added L11: 12 nH, Inductor_SMD:L_0603_1608Metric, symbol tx_board_symbol_library:L
- added L33: 12nH, Inductor_SMD:L_0603_1608Metric_Pad1.05x0.95mm_HandSolder, symbol Device:L
- added LNA0: PMA3-63GLN+, PMA3-63GLN+:QFN51P300X300X89-13N, symbol PMA3-63GLN+:PMA3-63GLN+
- added PA0: QPA9122TR7, QPA9122-TR7:QPA9122TR7, symbol tx_board_symbol_library:QPA9122TR7
- added PS0: MAPS-010164-TR0500, MAPS-010164-TR0500:QFN50P400X400X100-25N-D, symbol tx_board_symbol_library:MAPS-010164-TR0500
- added R12, R13, R14, R15, R16, R17, R33, R4: 50, Resistor_SMD:R_0402_1005Metric, symbol tx_board_symbol_library:R_US
- added R29: 8.2, Resistor_SMD:R_0402_1005Metric, symbol tx_board_symbol_library:R_US
- added R32: 51, Resistor_SMD:R_0402_1005Metric, symbol tx_board_symbol_library:R_US
- added R51, R52: 20k, Resistor_SMD:R_0402_1005Metric, symbol Device:R_US
- added SW00, SW01: PE42423B-Z, PE42423:QFN50P300X300X90-17N-D, symbol PE42423B-Z:PE42423B-Z
Connections:
- net AMP-RF_OUT: now also C50.2, SW01.11 (RF2)
- net ATTN-RF_OUT: now also AT0.9 (RFOUT), J8.1 (IN)
- net CLK: now also R12.1, R16.2
- net CPL_FWD: now also CPL0.10 (COUPLED_(FORWARD)), CPL_PORT0.1 (In)
- net GND: now also AT0.10 (GND_6), AT0.11 (GND_7), AT0.15 (A1), AT0.16 (A2), AT0.17 (EP), AT0.2 (A0), AT0.3 (GND_1), AT0.5 (GND_2), AT0.6 (GND_3), AT0.7 (GND_4), AT0.8 (GND_5), C1.2, C10.2, C11.1, C114.2, C115.2, C12.2, C129.1, C130.2, C141.1, C149.2, C2.1, C3.2, C36.2, C37.2, C38.2, C39.2, C40.1, C42.1, C43.2, C44.2, C45.1, C46.1, C47.2, C48.2, C49.2, C6.1, C7.2, C8.1, C9.1, CPL0.2 (GROUND_1), CPL0.3 (GROUND_2), CPL0.4 (GROUND_3), CPL0.7 (GROUND_4), CPL0.8 (GROUND_5), CPL0.9 (GROUND_6), CPL_PORT0.2 (Ext), J0.2, J0.3, J0.4, J0.5, J8.3 (GND_1), J8.4 (GND_2), LNA0.1 (NC_1), LNA0.10 (NC_8), LNA0.11 (NC_9), LNA0.12 (NC_10), LNA0.13 (EP), LNA0.3 (NC_2), LNA0.4 (NC_3), LNA0.5 (NC_4), LNA0.6 (NC_5), LNA0.7 (NC_6), LNA0.9 (NC_7), PA0.1 (NC_1), PA0.12 (NC_8), PA0.14 (NC_9), PA0.15 (NC_10), PA0.17 (GND), PA0.3 (NC_2), PA0.5 (NC_3), PA0.6 (NC_4), PA0.7 (NC_5), PA0.8 (NC_6), PA0.9 (NC_7), PS0.10 (GND_7), PS0.11 (GND_8), PS0.12 (GND_9), PS0.13 (GND_10), PS0.15 (GND_11), PS0.16 (GND_12), PS0.19 (D6), PS0.20 (D5), PS0.21 (D4), PS0.25 (EPAD), PS0.3 (GND_1), PS0.4 (GND_2), PS0.6 (GND_3), PS0.7 (GND_4), PS0.8 (GND_5), PS0.9 (GND_6), R33.2, R51.2, SW00.1 (GND_1), SW00.10 (GND_8), SW00.12 (GND_9), SW00.13 (GND_10), SW00.17 (GND_11), SW00.3 (GND_2), SW00.4 (GND_3), SW00.5 (GND_4), SW00.6 (GND_5), SW00.8 (GND_6), SW00.9 (GND_7), SW01.1 (GND_1), SW01.10 (GND_8), SW01.12 (GND_9), SW01.13 (GND_10), SW01.17 (GND_11), SW01.3 (GND_2), SW01.4 (GND_3), SW01.5 (GND_4), SW01.6 (GND_5), SW01.8 (GND_6), SW01.9 (GND_7)
- net OUTPUT: now also CPL0.6 (OUTPUT), J0.1
- net PS-RF_OUT: now also AT0.4 (RFIN), PS0.14 (RF_OUT)
- net SER_IN: now also R15.1, R4.1
- net SER_OUT: now also R14.1
- net TR_CTRL: now also C130.1, C149.1, SW00.14 (CTRL), SW01.14 (CTRL)
- net VCC: now also C1.1, C10.1, C114.1, C129.2, C141.2, C36.1, C44.1, C46.2, C47.1, C48.1, L1.1, L10.2, L2.1, L4.1, L6.1, L7.1, R32.1, R52.1, SW00.16 (VDD), SW01.16 (VDD)
- net VEE: now also C2.2, L3.1
- net V_PD: now also C42.2, L8.1
- new net: C11.2, L4.2, PS0.18 (VCC)
- new net: C9.2, PS0.22 (D3_OR_LE), R13.1
- new net: AT0.1 (VDD), C37.1, L6.2
- new net: C43.1, L7.2, R29.1
- new net: PA0.4 (VCC1/VCC2), R29.2
- new net: C50.1, L11.1, PA0.10 (RFOUT/VCC3_1), PA0.11 (RFOUT/VCC3_2)
- new net: C49.1, L10.1, L11.2
- new net: AT0.14 (SI), C38.1, R15.2
- new net: R52.2, SW01.15 (LS)
- new net: C113.1, SW01.2 (RF1)
- new net: CPL0.1 (INPUT), SW01.7 (RFC)
- new net: AT0.12 (LE), C40.2, R17.1
- new net: C113.2, LNA0.2 (RF-IN)
- new net: C116.1, L33.2, LNA0.8 (RF-OUT&DC-IN)
- new net: AT0.13 (CLK), C39.1, R16.1
- new net: C6.2, L3.2, PS0.1 (VEE)
- new net: C12.1, PS0.17 (SER_OUT), R14.2
- new net: C3.1, L2.2, PS0.2 (P/S)
- new net: C8.2, PS0.23 (D2_OR_CLK), R12.2
- new net: C7.1, PS0.24 (D1_OR_SER_IN), R4.2
- new net: J8.2 (OUT), SW00.7 (RFC)
- new net: R51.1, SW00.15 (LS)
- new net: PA0.13 (VBIAS), R32.2
- new net: C45.2, L8.2, PA0.16 (VPD)
- new net: C41.2, PA0.2 (RFIN)
- new net: C116.2, SW00.11 (RF2)
- new net: C115.1, L1.2, L33.1
- new net: CPL0.5 (COUPLED_(REVERSE)), R33.1
- new net: C41.1, SW00.2 (RF1)
- new net ATTN_LE_0: R17.2
- new net PS_LE_0: R13.2
- new net RF_IN_0: PS0.5 (RF_IN)
Other:
- note added: "very high cutoff LPFs to filter RF noise from power lines."
