File: Hardware/OpenPhasedArray0.3/channel0.kicad_sch (KiCad schematic)
At the start: 65 parts, among them J0 CONSMA022-G, J8 MM8030-2610RJ3, SW00 PE42423B-Z, SW01 PE42423B-Z

Commit message: better net naming
Connections:
- net VCC renamed +5VDC
- net VEE renamed -5VDC
- net V_PD renamed 1V8DC
Changed lines of the file:
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@@
 		)
 	)
-	(hierarchical_label "VCC"
+	(hierarchical_label "+5VDC"
 		(shape input)
 		(at 172.72 257.81 180)
@@
 		)
 	)
-	(hierarchical_label "VEE"
+	(hierarchical_label "-5VDC"
 		(shape input)
 		(at 187.96 255.27 180)
@@
 		)
 	)
-	(hierarchical_label "VCC"
+	(hierarchical_label "+5VDC"
 		(shape input)
 		(at 452.12 262.89 0)
@@
 		)
 	)
-	(hierarchical_label "V_PD"
+	(hierarchical_label "1V8DC"
 		(shape input)
 		(at 474.98 185.42 90)
@@
 		)
 	)
-	(hierarchical_label "VCC"
+	(hierarchical_label "+5VDC"
 		(shape input)
 		(at 246.38 227.33 90)
@@
 		)
 	)
-	(hierarchical_label "VCC"
+	(hierarchical_label "+5VDC"
 		(shape input)
 		(at 290.83 220.98 90)
@@
 		)
 	)
-	(hierarchical_label "VCC"
+	(hierarchical_label "+5VDC"
 		(shape input)
 		(at 530.86 177.8 90)
@@
 		)
 	)
-	(hierarchical_label "VCC"
+	(hierarchical_label "+5VDC"
 		(shape input)
 		(at 501.65 172.72 90)
@@
 		)
 	)
-	(hierarchical_label "VCC"
+	(hierarchical_label "+5VDC"
 		(shape input)
 		(at 480.06 331.47 0)
@@
 		)
 	)
-	(hierarchical_label "VCC"
+	(hierarchical_label "+5VDC"
 		(shape input)
 		(at 533.4 254 180)
@@
 		)
 	)
-	(hierarchical_label "VCC"
+	(hierarchical_label "+5VDC"
 		(shape input)
 		(at 529.59 251.46 180)
@@
 		)
 	)
-	(hierarchical_label "VCC"
+	(hierarchical_label "+5VDC"
 		(shape input)
 		(at 467.36 257.81 270)
