File: Hardware/OpenPhasedArray0.3/channel1.kicad_sch (KiCad schematic)
At the start: 65 parts, among them IC10 PE42423B-Z, IC6 MAPS-010164-TR0500, IC7 PE42423B-Z, IC8 QPA9122TR7, IC9 PMA3-63GLN+, J2 MM8030-2610RJ3, J4 CONSMA022-G, J7 Conn_Coaxial

Commit message: Restored broken Rev 2 for posterity and cleaned up naming
Parts:
- renumbered HY1 to CPL1, J7 to CPL_PORT1, J4 to J1, J2 to J9, IC9 to LNA1, IC8 to PA1, IC6 to PS1, IC7 to SW10, IC10 to SW11
Changed lines of the file:
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@@
 		(on_board yes)
 		(dnp no)
-		(property "Reference" "J2"
+		(property "Reference" "J9"
 			(at 410.972 296.926 90)
 			(effects
@@
 			(project "TX_Board_Rev2"
 				(path "/5327d041-dca0-47c6-802d-ce81714adf6c/1f7ad546-660a-419f-8ac2-791e37216311"
-					(reference "J2")
+					(reference "J9")
 					(unit 1)
 				)
@@
 		(on_board yes)
 		(dnp no)
-		(property "Reference" "IC6"
+		(property "Reference" "PS1"
 			(at 279.4 259.0098 0)
 			(effects
@@
 			(project "TX_Board_Rev2"
 				(path "/5327d041-dca0-47c6-802d-ce81714adf6c/1f7ad546-660a-419f-8ac2-791e37216311"
-					(reference "IC6")
+					(reference "PS1")
 					(unit 1)
 				)
@@
 		(dnp no)
 		(fields_autoplaced yes)
-		(property "Reference" "IC10"
+		(property "Reference" "SW11"
 			(at 587.4319 276.86 90)
 			(effects
@@
 			(project "TX_Board_Rev2"
 				(path "/5327d041-dca0-47c6-802d-ce81714adf6c/1f7ad546-660a-419f-8ac2-791e37216311"
-					(reference "IC10")
+					(reference "SW11")
 					(unit 1)
 				)
@@
 		(dnp no)
 		(fields_autoplaced yes)
-		(property "Reference" "IC8"
+		(property "Reference" "PA1"
 			(at 551.18 219.6398 0)
 			(effects
@@
 			(project "TX_Board_Rev2"
 				(path "/5327d041-dca0-47c6-802d-ce81714adf6c/1f7ad546-660a-419f-8ac2-791e37216311"
-					(reference "IC8")
+					(reference "PA1")
 					(unit 1)
 				)
@@
 		(on_board yes)
 		(dnp no)
-		(property "Reference" "IC9"
+		(property "Reference" "LNA1"
 			(at 531.622 313.436 0)
 			(effects
@@
 			(project "TX_Board_Rev2"
 				(path "/5327d041-dca0-47c6-802d-ce81714adf6c/1f7ad546-660a-419f-8ac2-791e37216311"
-					(reference "IC9")
+					(reference "LNA1")
 					(unit 1)
 				)
@@
 		(dnp no)
 		(fields_autoplaced yes)
-		(property "Reference" "J7"
+		(property "Reference" "CPL_PORT1"
 			(at 720.09 251.7531 0)
 			(effects
@@
 			(project "TX_Board_Rev2"
 				(path "/5327d041-dca0-47c6-802d-ce81714adf6c/1f7ad546-660a-419f-8ac2-791e37216311"
-					(reference "J7")
+					(reference "CPL_PORT1")
 					(unit 1)
 				)
@@
 		(dnp no)
 		(fields_autoplaced yes)
-		(property "Reference" "IC7"
+		(property "Reference" "SW10"
 			(at 456.5081 260.35 90)
 			(effects
@@
 			(project "TX_Board_Rev2"
 				(path "/5327d041-dca0-47c6-802d-ce81714adf6c/1f7ad546-660a-419f-8ac2-791e37216311"
-					(reference "IC7")
+					(reference "SW10")
 					(unit 1)
 				)
@@
 		(dnp no)
 		(fields_autoplaced yes)
-		(property "Reference" "HY1"
+		(property "Reference" "CPL1"
 			(at 670.56 254 0)
 			(effects
@@
 			(project "TX_Board_Rev2"
 				(path "/5327d041-dca0-47c6-802d-ce81714adf6c/1f7ad546-660a-419f-8ac2-791e37216311"
-					(reference "HY1")
+					(reference "CPL1")
 					(unit 1)
 				)
@@
 		(dnp no)
 		(fields_autoplaced yes)
-		(property "Reference" "J4"
+		(property "Reference" "J1"
 			(at 702.5005 273.05 0)
 			(effects
@@
 			(project "TX_Board_Rev2"
 				(path "/5327d041-dca0-47c6-802d-ce81714adf6c/1f7ad546-660a-419f-8ac2-791e37216311"
-					(reference "J4")
+					(reference "J1")
 					(unit 1)
 				)
