File: Hardware/OpenPhasedArray0.3/channel1.kicad_sch (KiCad schematic)
At the start: 65 parts, among them J1 CONSMA022-G, J9 MM8030-2610RJ3, SW10 PE42423B-Z, SW11 PE42423B-Z

Commit message: better net naming
Connections:
- net VCC renamed +5VDC
- net VEE renamed -5VDC
- net V_PD renamed 1V8DC
Changed lines of the file:
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@@
 		)
 	)
-	(hierarchical_label "VCC"
+	(hierarchical_label "+5VDC"
 		(shape input)
 		(at 201.93 267.97 180)
@@
 		)
 	)
-	(hierarchical_label "VCC"
+	(hierarchical_label "+5VDC"
 		(shape input)
 		(at 275.59 237.49 90)
@@
 		)
 	)
-	(hierarchical_label "V_PD"
+	(hierarchical_label "1V8DC"
 		(shape input)
 		(at 504.19 195.58 90)
@@
 		)
 	)
-	(hierarchical_label "VCC"
+	(hierarchical_label "+5VDC"
 		(shape input)
 		(at 481.33 273.05 0)
@@
 		)
 	)
-	(hierarchical_label "VCC"
+	(hierarchical_label "+5VDC"
 		(shape input)
 		(at 560.07 187.96 90)
@@
 		)
 	)
-	(hierarchical_label "VEE"
+	(hierarchical_label "-5VDC"
 		(shape input)
 		(at 217.17 265.43 180)
@@
 		)
 	)
-	(hierarchical_label "VCC"
+	(hierarchical_label "+5VDC"
 		(shape input)
 		(at 509.27 341.63 0)
@@
 		)
 	)
-	(hierarchical_label "VCC"
+	(hierarchical_label "+5VDC"
 		(shape input)
 		(at 496.57 267.97 270)
@@
 		)
 	)
-	(hierarchical_label "VCC"
+	(hierarchical_label "+5VDC"
 		(shape input)
 		(at 562.61 264.16 180)
@@
 		)
 	)
-	(hierarchical_label "VCC"
+	(hierarchical_label "+5VDC"
 		(shape input)
 		(at 320.04 231.14 90)
@@
 		)
 	)
-	(hierarchical_label "VCC"
+	(hierarchical_label "+5VDC"
 		(shape input)
 		(at 558.8 261.62 180)
@@
 		)
 	)
-	(hierarchical_label "VCC"
+	(hierarchical_label "+5VDC"
 		(shape input)
 		(at 530.86 182.88 90)
