File: Hardware/OpenPhasedArray0.3/channel2.kicad_sch (KiCad schematic)
At the start: 65 parts, among them IC10 PE42423B-Z, IC6 MAPS-010164-TR0500, IC7 PE42423B-Z, IC8 QPA9122TR7, IC9 PMA3-63GLN+, J2 MM8030-2610RJ3, J4 CONSMA022-G, J7 Conn_Coaxial

Commit message: Restored broken Rev 2 for posterity and cleaned up naming
Parts:
- removed AT1: RFSA3713TR7, RFSA3713:QFN50P300X300X90-17N, symbol tx_board_symbol_library:RFSA3713TR7
- removed C13, C14, C20: 0.1uF, Capacitor_SMD:C_0402_1005Metric, symbol tx_board_symbol_library:C
- removed C15, C16, C21: 100pF, Capacitor_SMD:C_0402_1005Metric, symbol tx_board_symbol_library:C
- removed C17, C18, C19, C22, C25, C26, C27: 1.3 pF, Capacitor_SMD:C_0402_1005Metric, symbol tx_board_symbol_library:C
- removed C23: 470p, Capacitor_SMD:C_0402_1005Metric, symbol tx_board_symbol_library:C
- removed C24: 1uF, Capacitor_SMD:C_0402_1005Metric, symbol tx_board_symbol_library:C
- removed C28, C29, C56, C57: 22 pF, Capacitor_SMD:C_0402_1005Metric, symbol Device:C_Small
- removed C30, C60: 18 pF, Capacitor_SMD:C_0402_1005Metric, symbol tx_board_symbol_library:C
- removed C31, C55: 18pF, Capacitor_SMD:C_0402_1005Metric, symbol Device:C
- removed C32, C34, C58: 1 uF, Capacitor_SMD:C_0402_1005Metric, symbol tx_board_symbol_library:C
- removed C33, C52, C53, C54, C59: 100 pF, Capacitor_SMD:C_0402_1005Metric, symbol tx_board_symbol_library:C
- removed C35: 100pF, Capacitor_SMD:C_0402_1005Metric, symbol Device:C
- removed C51: 10uF, Capacitor_SMD:C_0402_1005Metric, symbol Device:C
- removed HY1: BDCA1-10-40+, BDCA1-10-40+:BDCA11040, symbol BDCA1-10-40+:BDCA1-10-40+
- removed IC10, IC7: PE42423B-Z, PE42423:QFN50P300X300X90-17N-D, symbol PE42423B-Z:PE42423B-Z
- removed IC6: MAPS-010164-TR0500, MAPS-010164-TR0500:QFN50P400X400X100-25N-D, symbol tx_board_symbol_library:MAPS-010164-TR0500
- removed IC8: QPA9122TR7, QPA9122-TR7:QPA9122TR7, symbol tx_board_symbol_library:QPA9122TR7
- removed IC9: PMA3-63GLN+, PMA3-63GLN+:QFN51P300X300X89-13N, symbol PMA3-63GLN+:PMA3-63GLN+
- removed J2: MM8030-2610RJ3, MM8030-2610RJ3:MM80302610RJ3, symbol tx_board_symbol_library:MM8030-2610RJ3
- removed J4: CONSMA022-G, CONSMA022_G:LINX_CONSMA022-G, symbol CONSMA022-G:CONSMA022-G
- removed J7: Conn_Coaxial, Connector_Coaxial:SMA_Amphenol_901-144_Vertical, symbol Connector:Conn_Coaxial
- removed L12, L13, L14, L15, L17, L18, L5, L9: L_Ferrite, Inductor_SMD:L_0201_0603Metric_Pad0.64x0.40mm_HandSolder, symbol Device:L_Ferrite
- removed L16: 12nH, Inductor_SMD:L_0603_1608Metric_Pad1.05x0.95mm_HandSolder, symbol Device:L
- removed L19: 12 nH, Inductor_SMD:L_0603_1608Metric, symbol tx_board_symbol_library:L
- removed R18, R19, R20, R21, R22, R23, R24, R27: 50, Resistor_SMD:R_0402_1005Metric, symbol tx_board_symbol_library:R_US
- removed R25: 8.2, Resistor_SMD:R_0402_1005Metric, symbol tx_board_symbol_library:R_US
- removed R26: 51, Resistor_SMD:R_0402_1005Metric, symbol tx_board_symbol_library:R_US
- removed R53, R54: 20k, Resistor_SMD:R_0402_1005Metric, symbol Device:R_US
- added AT2: RFSA3713TR7, RFSA3713:QFN50P300X300X90-17N, symbol tx_board_symbol_library:RFSA3713TR7
- added C61, C62, C68: 0.1uF, Capacitor_SMD:C_0402_1005Metric, symbol tx_board_symbol_library:C
- added C63, C64, C69: 100pF, Capacitor_SMD:C_0402_1005Metric, symbol tx_board_symbol_library:C
- added C65, C66, C67, C70, C73, C74, C75: 1.3 pF, Capacitor_SMD:C_0402_1005Metric, symbol tx_board_symbol_library:C
- added C71: 470p, Capacitor_SMD:C_0402_1005Metric, symbol tx_board_symbol_library:C
- added C72: 1uF, Capacitor_SMD:C_0402_1005Metric, symbol tx_board_symbol_library:C
- added C76, C77, C89, C90: 22 pF, Capacitor_SMD:C_0402_1005Metric, symbol Device:C_Small
- added C78, C93: 18 pF, Capacitor_SMD:C_0402_1005Metric, symbol tx_board_symbol_library:C
- added C79, C88: 18pF, Capacitor_SMD:C_0402_1005Metric, symbol Device:C
- added C80, C82, C91: 1 uF, Capacitor_SMD:C_0402_1005Metric, symbol tx_board_symbol_library:C
- added C81, C85, C86, C87, C92: 100 pF, Capacitor_SMD:C_0402_1005Metric, symbol tx_board_symbol_library:C
- added C83: 100pF, Capacitor_SMD:C_0402_1005Metric, symbol Device:C
- added C84: 10uF, Capacitor_SMD:C_0402_1005Metric, symbol Device:C
- added CPL2: BDCA1-10-40+, BDCA1-10-40+:BDCA11040, symbol BDCA1-10-40+:BDCA1-10-40+
- added CPL_PORT2: Conn_Coaxial, Connector_Coaxial:SMA_Amphenol_901-144_Vertical, symbol Connector:Conn_Coaxial
- added J10: MM8030-2610RJ3, MM8030-2610RJ3:MM80302610RJ3, symbol tx_board_symbol_library:MM8030-2610RJ3
- added J2: CONSMA022-G, CONSMA022_G:LINX_CONSMA022-G, symbol CONSMA022-G:CONSMA022-G
- added L20, L21, L22, L23, L24, L25, L27, L28: L_Ferrite, Inductor_SMD:L_0201_0603Metric_Pad0.64x0.40mm_HandSolder, symbol Device:L_Ferrite
- added L26: 12nH, Inductor_SMD:L_0603_1608Metric_Pad1.05x0.95mm_HandSolder, symbol Device:L
- added L29: 12 nH, Inductor_SMD:L_0603_1608Metric, symbol tx_board_symbol_library:L
- added LNA2: PMA3-63GLN+, PMA3-63GLN+:QFN51P300X300X89-13N, symbol PMA3-63GLN+:PMA3-63GLN+
- added PA2: QPA9122TR7, QPA9122-TR7:QPA9122TR7, symbol tx_board_symbol_library:QPA9122TR7
- added PS2: MAPS-010164-TR0500, MAPS-010164-TR0500:QFN50P400X400X100-25N-D, symbol tx_board_symbol_library:MAPS-010164-TR0500
- added R28, R30, R31, R34, R35, R36, R37, R40: 50, Resistor_SMD:R_0402_1005Metric, symbol tx_board_symbol_library:R_US
- added R38: 8.2, Resistor_SMD:R_0402_1005Metric, symbol tx_board_symbol_library:R_US
- added R39: 51, Resistor_SMD:R_0402_1005Metric, symbol tx_board_symbol_library:R_US
- added R55, R56: 20k, Resistor_SMD:R_0402_1005Metric, symbol Device:R_US
- added SW20, SW21: PE42423B-Z, PE42423:QFN50P300X300X90-17N-D, symbol PE42423B-Z:PE42423B-Z
Connections:
- net AMP-RF_OUT: now also C93.2, SW21.11 (RF2)
- net ATTN-RF_OUT: now also AT2.9 (RFOUT), J10.1 (IN)
- net CLK: now also R30.1, R36.2
- net CPL_FWD: now also CPL2.10 (COUPLED_(FORWARD)), CPL_PORT2.1 (In)
- net GND: now also AT2.10 (GND_6), AT2.11 (GND_7), AT2.15 (A1), AT2.16 (A2), AT2.17 (EP), AT2.2 (A0), AT2.3 (GND_1), AT2.5 (GND_2), AT2.6 (GND_3), AT2.7 (GND_4), AT2.8 (GND_5), C61.2, C62.1, C63.2, C64.1, C65.2, C66.1, C67.1, C68.2, C69.1, C70.2, C71.2, C72.2, C73.2, C74.2, C75.1, C76.1, C77.2, C80.1, C81.2, C82.2, C83.2, C84.2, C85.1, C86.1, C87.2, C89.2, C90.1, C91.2, C92.2, CPL2.2 (GROUND_1), CPL2.3 (GROUND_2), CPL2.4 (GROUND_3), CPL2.7 (GROUND_4), CPL2.8 (GROUND_5), CPL2.9 (GROUND_6), CPL_PORT2.2 (Ext), J10.3 (GND_1), J10.4 (GND_2), J2.2, J2.3, J2.4, J2.5, LNA2.1 (NC_1), LNA2.10 (NC_8), LNA2.11 (NC_9), LNA2.12 (NC_10), LNA2.13 (EP), LNA2.3 (NC_2), LNA2.4 (NC_3), LNA2.5 (NC_4), LNA2.6 (NC_5), LNA2.7 (NC_6), LNA2.9 (NC_7), PA2.1 (NC_1), PA2.12 (NC_8), PA2.14 (NC_9), PA2.15 (NC_10), PA2.17 (GND), PA2.3 (NC_2), PA2.5 (NC_3), PA2.6 (NC_4), PA2.7 (NC_5), PA2.8 (NC_6), PA2.9 (NC_7), PS2.10 (GND_7), PS2.11 (GND_8), PS2.12 (GND_9), PS2.13 (GND_10), PS2.15 (GND_11), PS2.16 (GND_12), PS2.19 (D6), PS2.20 (D5), PS2.21 (D4), PS2.25 (EPAD), PS2.3 (GND_1), PS2.4 (GND_2), PS2.6 (GND_3), PS2.7 (GND_4), PS2.8 (GND_5), PS2.9 (GND_6), R40.2, R55.2, SW20.1 (GND_1), SW20.10 (GND_8), SW20.12 (GND_9), SW20.13 (GND_10), SW20.17 (GND_11), SW20.3 (GND_2), SW20.4 (GND_3), SW20.5 (GND_4), SW20.6 (GND_5), SW20.8 (GND_6), SW20.9 (GND_7), SW21.1 (GND_1), SW21.10 (GND_8), SW21.12 (GND_9), SW21.13 (GND_10), SW21.17 (GND_11), SW21.3 (GND_2), SW21.4 (GND_3), SW21.5 (GND_4), SW21.6 (GND_5), SW21.8 (GND_6), SW21.9 (GND_7)
- net OUTPUT: now also CPL2.6 (OUTPUT), J2.1
- net PS-RF_OUT: now also AT2.4 (RFIN), PS2.14 (RF_OUT)
- net SER_IN: now also R28.1, R35.1
- net SER_OUT: now also R34.1
- net TR_CTRL: now also C77.1, C89.1, SW20.14 (CTRL), SW21.14 (CTRL)
- net VCC: now also C61.1, C68.1, C71.1, C76.2, C82.1, C84.1, C86.2, C87.1, C90.2, C91.1, L20.1, L22.1, L23.1, L24.1, L27.1, L28.2, R39.1, R56.1, SW20.16 (VDD), SW21.16 (VDD)
- net VEE: now also C62.2, L21.1
- net V_PD: now also C80.2, L25.1
- new net: C85.2, L25.2, PA2.16 (VPD)
- new net: C88.2, LNA2.2 (RF-IN)
- new net: C79.1, L26.2, LNA2.8 (RF-OUT&DC-IN)
- new net: C66.2, PS2.23 (D2_OR_CLK), R30.2
- new net: C64.2, L21.2, PS2.1 (VEE)
- new net: CPL2.5 (COUPLED_(REVERSE)), R40.1
- new net: C65.1, PS2.24 (D1_OR_SER_IN), R28.2
- new net: C63.1, L20.2, PS2.2 (P/S)
- new net: CPL2.1 (INPUT), SW21.7 (RFC)
- new net: C69.2, L22.2, PS2.18 (VCC)
- new net: C67.2, PS2.22 (D3_OR_LE), R31.1
- new net: C93.1, L29.1, PA2.10 (RFOUT/VCC3_1), PA2.11 (RFOUT/VCC3_2)
- new net: R56.2, SW21.15 (LS)
- new net: C88.1, SW21.2 (RF1)
- new net: C70.1, PS2.17 (SER_OUT), R34.2
- new net: AT2.13 (CLK), C74.1, R36.1
- new net: AT2.1 (VDD), C72.1, L23.2
- new net: AT2.12 (LE), C75.2, R37.1
- new net: AT2.14 (SI), C73.1, R35.2
- new net: C92.1, L28.1, L29.2
- new net: C81.1, L24.2, R38.1
- new net: PA2.4 (VCC1/VCC2), R38.2
- new net: PA2.13 (VBIAS), R39.2
- new net: C78.2, PA2.2 (RFIN)
- new net: C79.2, SW20.11 (RF2)
- new net: C83.1, L26.1, L27.2
- new net: C78.1, SW20.2 (RF1)
- new net: J10.2 (OUT), SW20.7 (RFC)
- new net: R55.1, SW20.15 (LS)
- new net ATTN_LE_2: R37.2
- new net PS_LE_2: R31.2
- new net RF_IN_2: PS2.5 (RF_IN)
