File: Hardware/OpenPhasedArray0.3/channel2.kicad_sch (KiCad schematic)
At the start: 65 parts, among them J10 MM8030-2610RJ3, J2 CONSMA022-G, SW20 PE42423B-Z, SW21 PE42423B-Z

Commit message: better net naming
Connections:
- net VCC renamed +5VDC
- net VEE renamed -5VDC
- net V_PD renamed 1V8DC
Changed lines of the file:
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@@
 		)
 	)
-	(hierarchical_label "VCC"
+	(hierarchical_label "+5VDC"
 		(shape input)
 		(at 528.32 354.33 0)
@@
 		)
 	)
-	(hierarchical_label "VCC"
+	(hierarchical_label "+5VDC"
 		(shape input)
 		(at 581.66 276.86 180)
@@
 		)
 	)
-	(hierarchical_label "VCC"
+	(hierarchical_label "+5VDC"
 		(shape input)
 		(at 577.85 274.32 180)
@@
 		)
 	)
-	(hierarchical_label "VCC"
+	(hierarchical_label "+5VDC"
 		(shape input)
 		(at 294.64 250.19 90)
@@
 		)
 	)
-	(hierarchical_label "VCC"
+	(hierarchical_label "+5VDC"
 		(shape input)
 		(at 220.98 280.67 180)
@@
 		)
 	)
-	(hierarchical_label "VEE"
+	(hierarchical_label "-5VDC"
 		(shape input)
 		(at 236.22 278.13 180)
@@
 		)
 	)
-	(hierarchical_label "VCC"
+	(hierarchical_label "+5VDC"
 		(shape input)
 		(at 579.12 200.66 90)
@@
 		)
 	)
-	(hierarchical_label "V_PD"
+	(hierarchical_label "1V8DC"
 		(shape input)
 		(at 523.24 208.28 90)
@@
 		)
 	)
-	(hierarchical_label "VCC"
+	(hierarchical_label "+5VDC"
 		(shape input)
 		(at 515.62 280.67 270)
@@
 		)
 	)
-	(hierarchical_label "VCC"
+	(hierarchical_label "+5VDC"
 		(shape input)
 		(at 339.09 243.84 90)
@@
 		)
 	)
-	(hierarchical_label "VCC"
+	(hierarchical_label "+5VDC"
 		(shape input)
 		(at 500.38 285.75 0)
@@
 		)
 	)
-	(hierarchical_label "VCC"
+	(hierarchical_label "+5VDC"
 		(shape input)
 		(at 549.91 195.58 90)
