File: Hardware/OpenPhasedArray0.3/channel3.kicad_sch (KiCad schematic)
At the start: 65 parts, among them IC10 PE42423B-Z, IC6 MAPS-010164-TR0500, IC7 PE42423B-Z, IC8 QPA9122TR7, IC9 PMA3-63GLN+, J2 MM8030-2610RJ3, J4 CONSMA022-G, J7 Conn_Coaxial

Commit message: Restored broken Rev 2 for posterity and cleaned up naming
Parts:
- removed AT1: RFSA3713TR7, RFSA3713:QFN50P300X300X90-17N, symbol tx_board_symbol_library:RFSA3713TR7
- removed C13, C14, C20: 0.1uF, Capacitor_SMD:C_0402_1005Metric, symbol tx_board_symbol_library:C
- removed C15, C16, C21: 100pF, Capacitor_SMD:C_0402_1005Metric, symbol tx_board_symbol_library:C
- removed C17, C18, C19, C22, C25, C26, C27: 1.3 pF, Capacitor_SMD:C_0402_1005Metric, symbol tx_board_symbol_library:C
- removed C23: 470p, Capacitor_SMD:C_0402_1005Metric, symbol tx_board_symbol_library:C
- removed C24: 1uF, Capacitor_SMD:C_0402_1005Metric, symbol tx_board_symbol_library:C
- removed C28, C29, C56, C57: 22 pF, Capacitor_SMD:C_0402_1005Metric, symbol Device:C_Small
- removed C30, C60: 18 pF, Capacitor_SMD:C_0402_1005Metric, symbol tx_board_symbol_library:C
- removed C31, C55: 18pF, Capacitor_SMD:C_0402_1005Metric, symbol Device:C
- removed C32, C34, C58: 1 uF, Capacitor_SMD:C_0402_1005Metric, symbol tx_board_symbol_library:C
- removed C33, C52, C53, C54, C59: 100 pF, Capacitor_SMD:C_0402_1005Metric, symbol tx_board_symbol_library:C
- removed C35: 100pF, Capacitor_SMD:C_0402_1005Metric, symbol Device:C
- removed C51: 10uF, Capacitor_SMD:C_0402_1005Metric, symbol Device:C
- removed HY1: BDCA1-10-40+, BDCA1-10-40+:BDCA11040, symbol BDCA1-10-40+:BDCA1-10-40+
- removed IC10, IC7: PE42423B-Z, PE42423:QFN50P300X300X90-17N-D, symbol PE42423B-Z:PE42423B-Z
- removed IC6: MAPS-010164-TR0500, MAPS-010164-TR0500:QFN50P400X400X100-25N-D, symbol tx_board_symbol_library:MAPS-010164-TR0500
- removed IC8: QPA9122TR7, QPA9122-TR7:QPA9122TR7, symbol tx_board_symbol_library:QPA9122TR7
- removed IC9: PMA3-63GLN+, PMA3-63GLN+:QFN51P300X300X89-13N, symbol PMA3-63GLN+:PMA3-63GLN+
- removed J2: MM8030-2610RJ3, MM8030-2610RJ3:MM80302610RJ3, symbol tx_board_symbol_library:MM8030-2610RJ3
- removed J4: CONSMA022-G, CONSMA022_G:LINX_CONSMA022-G, symbol CONSMA022-G:CONSMA022-G
- removed J7: Conn_Coaxial, Connector_Coaxial:SMA_Amphenol_901-144_Vertical, symbol Connector:Conn_Coaxial
- removed L12, L13, L14, L15, L17, L18, L5, L9: L_Ferrite, Inductor_SMD:L_0201_0603Metric_Pad0.64x0.40mm_HandSolder, symbol Device:L_Ferrite
- removed L16: 12nH, Inductor_SMD:L_0603_1608Metric_Pad1.05x0.95mm_HandSolder, symbol Device:L
- removed L19: 12 nH, Inductor_SMD:L_0603_1608Metric, symbol tx_board_symbol_library:L
- removed R18, R19, R20, R21, R22, R23, R24, R27: 50, Resistor_SMD:R_0402_1005Metric, symbol tx_board_symbol_library:R_US
- removed R25: 8.2, Resistor_SMD:R_0402_1005Metric, symbol tx_board_symbol_library:R_US
- removed R26: 51, Resistor_SMD:R_0402_1005Metric, symbol tx_board_symbol_library:R_US
- removed R53, R54: 20k, Resistor_SMD:R_0402_1005Metric, symbol Device:R_US
- added AT3: RFSA3713TR7, RFSA3713:QFN50P300X300X90-17N, symbol tx_board_symbol_library:RFSA3713TR7
- added C100, C103, C106, C107, C108, C98, C99: 1.3 pF, Capacitor_SMD:C_0402_1005Metric, symbol tx_board_symbol_library:C
- added C101, C94, C95: 0.1uF, Capacitor_SMD:C_0402_1005Metric, symbol tx_board_symbol_library:C
- added C102, C96, C97: 100pF, Capacitor_SMD:C_0402_1005Metric, symbol tx_board_symbol_library:C
- added C104: 470p, Capacitor_SMD:C_0402_1005Metric, symbol tx_board_symbol_library:C
- added C105: 1uF, Capacitor_SMD:C_0402_1005Metric, symbol tx_board_symbol_library:C
- added C109, C110, C126, C127: 22 pF, Capacitor_SMD:C_0402_1005Metric, symbol Device:C_Small
- added C111, C132: 18 pF, Capacitor_SMD:C_0402_1005Metric, symbol tx_board_symbol_library:C
- added C112, C125: 18pF, Capacitor_SMD:C_0402_1005Metric, symbol Device:C
- added C117, C119, C128: 1 uF, Capacitor_SMD:C_0402_1005Metric, symbol tx_board_symbol_library:C
- added C118, C122, C123, C124, C131: 100 pF, Capacitor_SMD:C_0402_1005Metric, symbol tx_board_symbol_library:C
- added C120: 100pF, Capacitor_SMD:C_0402_1005Metric, symbol Device:C
- added C121: 10uF, Capacitor_SMD:C_0402_1005Metric, symbol Device:C
- added CPL3: BDCA1-10-40+, BDCA1-10-40+:BDCA11040, symbol BDCA1-10-40+:BDCA1-10-40+
- added CPL_PORT3: Conn_Coaxial, Connector_Coaxial:SMA_Amphenol_901-144_Vertical, symbol Connector:Conn_Coaxial
- added J11: MM8030-2610RJ3, MM8030-2610RJ3:MM80302610RJ3, symbol tx_board_symbol_library:MM8030-2610RJ3
- added J3: CONSMA022-G, CONSMA022_G:LINX_CONSMA022-G, symbol CONSMA022-G:CONSMA022-G
- added L30, L31, L32, L34, L35, L36, L38, L39: L_Ferrite, Inductor_SMD:L_0201_0603Metric_Pad0.64x0.40mm_HandSolder, symbol Device:L_Ferrite
- added L37: 12nH, Inductor_SMD:L_0603_1608Metric_Pad1.05x0.95mm_HandSolder, symbol Device:L
- added L40: 12 nH, Inductor_SMD:L_0603_1608Metric, symbol tx_board_symbol_library:L
- added LNA3: PMA3-63GLN+, PMA3-63GLN+:QFN51P300X300X89-13N, symbol PMA3-63GLN+:PMA3-63GLN+
- added PA3: QPA9122TR7, QPA9122-TR7:QPA9122TR7, symbol tx_board_symbol_library:QPA9122TR7
- added PS3: MAPS-010164-TR0500, MAPS-010164-TR0500:QFN50P400X400X100-25N-D, symbol tx_board_symbol_library:MAPS-010164-TR0500
- added R41, R42, R43, R44, R45, R46, R47, R50: 50, Resistor_SMD:R_0402_1005Metric, symbol tx_board_symbol_library:R_US
- added R48: 8.2, Resistor_SMD:R_0402_1005Metric, symbol tx_board_symbol_library:R_US
- added R49: 51, Resistor_SMD:R_0402_1005Metric, symbol tx_board_symbol_library:R_US
- added R57, R58: 20k, Resistor_SMD:R_0402_1005Metric, symbol Device:R_US
- added SW30, SW31: PE42423B-Z, PE42423:QFN50P300X300X90-17N-D, symbol PE42423B-Z:PE42423B-Z
Connections:
- net AMP-RF_OUT: now also C132.2, SW31.11 (RF2)
- net ATTN-RF_OUT: now also AT3.9 (RFOUT), J11.1 (IN)
- net CLK: now also R42.1, R46.2
- net CPL_FWD: now also CPL3.10 (COUPLED_(FORWARD)), CPL_PORT3.1 (In)
- net GND: now also AT3.10 (GND_6), AT3.11 (GND_7), AT3.15 (A1), AT3.16 (A2), AT3.17 (EP), AT3.2 (A0), AT3.3 (GND_1), AT3.5 (GND_2), AT3.6 (GND_3), AT3.7 (GND_4), AT3.8 (GND_5), C100.1, C101.2, C102.1, C103.2, C104.2, C105.2, C106.2, C107.2, C108.1, C109.1, C110.2, C117.1, C118.2, C119.2, C120.2, C121.2, C122.1, C123.1, C124.2, C126.2, C127.1, C128.2, C131.2, C94.2, C95.1, C96.2, C97.1, C98.2, C99.1, CPL3.2 (GROUND_1), CPL3.3 (GROUND_2), CPL3.4 (GROUND_3), CPL3.7 (GROUND_4), CPL3.8 (GROUND_5), CPL3.9 (GROUND_6), CPL_PORT3.2 (Ext), J11.3 (GND_1), J11.4 (GND_2), J3.2, J3.3, J3.4, J3.5, LNA3.1 (NC_1), LNA3.10 (NC_8), LNA3.11 (NC_9), LNA3.12 (NC_10), LNA3.13 (EP), LNA3.3 (NC_2), LNA3.4 (NC_3), LNA3.5 (NC_4), LNA3.6 (NC_5), LNA3.7 (NC_6), LNA3.9 (NC_7), PA3.1 (NC_1), PA3.12 (NC_8), PA3.14 (NC_9), PA3.15 (NC_10), PA3.17 (GND), PA3.3 (NC_2), PA3.5 (NC_3), PA3.6 (NC_4), PA3.7 (NC_5), PA3.8 (NC_6), PA3.9 (NC_7), PS3.10 (GND_7), PS3.11 (GND_8), PS3.12 (GND_9), PS3.13 (GND_10), PS3.15 (GND_11), PS3.16 (GND_12), PS3.19 (D6), PS3.20 (D5), PS3.21 (D4), PS3.25 (EPAD), PS3.3 (GND_1), PS3.4 (GND_2), PS3.6 (GND_3), PS3.7 (GND_4), PS3.8 (GND_5), PS3.9 (GND_6), R50.2, R57.2, SW30.1 (GND_1), SW30.10 (GND_8), SW30.12 (GND_9), SW30.13 (GND_10), SW30.17 (GND_11), SW30.3 (GND_2), SW30.4 (GND_3), SW30.5 (GND_4), SW30.6 (GND_5), SW30.8 (GND_6), SW30.9 (GND_7), SW31.1 (GND_1), SW31.10 (GND_8), SW31.12 (GND_9), SW31.13 (GND_10), SW31.17 (GND_11), SW31.3 (GND_2), SW31.4 (GND_3), SW31.5 (GND_4), SW31.6 (GND_5), SW31.8 (GND_6), SW31.9 (GND_7)
- net OUTPUT: now also CPL3.6 (OUTPUT), J3.1
- net PS-RF_OUT: now also AT3.4 (RFIN), PS3.14 (RF_OUT)
- net SER_IN: now also R41.1, R45.1
- net SER_OUT: now also R44.1
- net TR_CTRL: now also C110.1, C126.1, SW30.14 (CTRL), SW31.14 (CTRL)
- net VCC: now also C101.1, C104.1, C109.2, C119.1, C121.1, C123.2, C124.1, C127.2, C128.1, C94.1, L30.1, L32.1, L34.1, L35.1, L38.1, L39.2, R49.1, R58.1, SW30.16 (VDD), SW31.16 (VDD)
- net VEE: now also C95.2, L31.1
- net V_PD: now also C117.2, L36.1
- new net: C120.1, L37.1, L38.2
- new net: C112.1, L37.2, LNA3.8 (RF-OUT&DC-IN)
- new net: C132.1, L40.1, PA3.10 (RFOUT/VCC3_1), PA3.11 (RFOUT/VCC3_2)
- new net: PA3.13 (VBIAS), R49.2
- new net: C122.2, L36.2, PA3.16 (VPD)
- new net: C111.2, PA3.2 (RFIN)
- new net: PA3.4 (VCC1/VCC2), R48.2
- new net: C112.2, SW30.11 (RF2)
- new net: C103.1, PS3.17 (SER_OUT), R44.2
- new net: R57.1, SW30.15 (LS)
- new net: C111.1, SW30.2 (RF1)
- new net: J11.2 (OUT), SW30.7 (RFC)
- new net: C100.2, PS3.22 (D3_OR_LE), R43.1
- new net: C96.1, L30.2, PS3.2 (P/S)
- new net: AT3.12 (LE), C108.2, R47.1
- new net: CPL3.1 (INPUT), SW31.7 (RFC)
- new net: CPL3.5 (COUPLED_(REVERSE)), R50.1
- new net: C98.1, PS3.24 (D1_OR_SER_IN), R41.2
- new net: C131.1, L39.1, L40.2
- new net: AT3.13 (CLK), C107.1, R46.1
- new net: AT3.1 (VDD), C105.1, L34.2
- new net: C97.2, L31.2, PS3.1 (VEE)
- new net: C118.1, L35.2, R48.1
- new net: AT3.14 (SI), C106.1, R45.2
- new net: C125.2, LNA3.2 (RF-IN)
- new net: R58.2, SW31.15 (LS)
- new net: C102.2, L32.2, PS3.18 (VCC)
- new net: C99.2, PS3.23 (D2_OR_CLK), R42.2
- new net: C125.1, SW31.2 (RF1)
- new net ATTN_LE_3: R47.2
- new net PS_LE_3: R43.2
- new net RF_IN_3: PS3.5 (RF_IN)
