File: Hardware/OpenPhasedArray0.3/channel3.kicad_sch (KiCad schematic)
At the start: 65 parts, among them J11 MM8030-2610RJ3, J3 CONSMA022-G, SW30 PE42423B-Z, SW31 PE42423B-Z

Commit message: better net naming
Connections:
- net VCC renamed +5VDC
- net VEE renamed -5VDC
- net V_PD renamed 1V8DC
Changed lines of the file:
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@@
 		)
 	)
-	(hierarchical_label "VCC"
+	(hierarchical_label "+5VDC"
 		(shape input)
 		(at 464.82 302.26 0)
@@
 		)
 	)
-	(hierarchical_label "VCC"
+	(hierarchical_label "+5VDC"
 		(shape input)
 		(at 303.53 260.35 90)
@@
 		)
 	)
-	(hierarchical_label "VCC"
+	(hierarchical_label "+5VDC"
 		(shape input)
 		(at 514.35 212.09 90)
@@
 		)
 	)
-	(hierarchical_label "VCC"
+	(hierarchical_label "+5VDC"
 		(shape input)
 		(at 542.29 290.83 180)
@@
 		)
 	)
-	(hierarchical_label "VCC"
+	(hierarchical_label "+5VDC"
 		(shape input)
 		(at 259.08 266.7 90)
@@
 		)
 	)
-	(hierarchical_label "VCC"
+	(hierarchical_label "+5VDC"
 		(shape input)
 		(at 543.56 217.17 90)
@@
 		)
 	)
-	(hierarchical_label "VEE"
+	(hierarchical_label "-5VDC"
 		(shape input)
 		(at 200.66 294.64 180)
@@
 		)
 	)
-	(hierarchical_label "VCC"
+	(hierarchical_label "+5VDC"
 		(shape input)
 		(at 492.76 370.84 0)
@@
 		)
 	)
-	(hierarchical_label "V_PD"
+	(hierarchical_label "1V8DC"
 		(shape input)
 		(at 487.68 224.79 90)
@@
 		)
 	)
-	(hierarchical_label "VCC"
+	(hierarchical_label "+5VDC"
 		(shape input)
 		(at 546.1 293.37 180)
@@
 		)
 	)
-	(hierarchical_label "VCC"
+	(hierarchical_label "+5VDC"
 		(shape input)
 		(at 185.42 297.18 180)
@@
 		)
 	)
-	(hierarchical_label "VCC"
+	(hierarchical_label "+5VDC"
 		(shape input)
 		(at 480.06 297.18 270)
