File: Hardware/OpenPhasedArray0.3/TX_Board_Rev2.kicad_sch (KiCad schematic)
At the start: 57 parts, among them IC1 GP2Y1+, IC2 GP2Y1+, IC3 GP2Y1+, J18 Conn_01x08, J19 694106301002, J4 MM8030-2610RJ3, J5 MM8030-2610RJ3, J6 MM8030-2610RJ3, J7 MM8030-2610RJ3, U1 SN74HCT138NSR, U2 SN74AHCT125DGVR

Commit message: clarified schematic comments, shrunk vias in QFN pads
Other:
- note added: "According to data sheet, unused inputs must be pulled high or low. It is CRITICAL that the SPI clock behavior be set in stone before assembly. Resistors to pull up and down are specced on both lines, but one MUST be D.N.P'ed before fab/assembly SPI Mode 0 or 1 -- keep the CLK pull-down SPI Mode 2 or 3 -- keep the CLK pull-up"
- note added: "It is technically possible to swap these resistors after fab but their layout will make you not want to"
- note removed: "According to data sheet, unused inputs must be pulled high or low. It is CRITICAL that the SPI clock behavior be set in stone before assembly. Resistors to pull up and down are specced on both lines, but one MUST be D.N.P'ed before fab/assembly SPI Mode 0 or 1 -- keep the pull-down SPI Mode 2 or 3 -- keep the pull-up"
Changed lines of the file:
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@@
 		)
 	)
-	(text "According to data sheet, \nunused inputs must be pulled \nhigh or low. It is CRITICAL that\nthe SPI clock behavior be set in stone\nbefore assembly. Resistors to pull up and \ndown are specced on both lines, but one\nMUST be D.N.P'ed before fab/assembly\n\nSPI Mode 0 or 1 -- keep the pull-down\nSPI Mode 2 or 3 -- keep the pull-up"
+	(text "According to data sheet, \nunused inputs must be pulled \nhigh or low. It is CRITICAL that\nthe SPI clock behavior be set in stone\nbefore assembly. Resistors to pull up and \ndown are specced on both lines, but one\nMUST be D.N.P'ed before fab/assembly\n\nSPI Mode 0 or 1 -- keep the CLK pull-down\nSPI Mode 2 or 3 -- keep the CLK pull-up"
 		(exclude_from_sim no)
-		(at 333.756 326.898 0)
+		(at 325.374 326.644 0)
 		(effects
 			(font
@@
 			)
 		)
+	)
+	(text "It is technically possible to swap \nthese resistors after fab but their \nlayout will make you not want to"
+		(exclude_from_sim no)
+		(at 327.66 375.412 0)
+		(effects
+			(font
+				(size 1.27 1.27)
+			)
+		)

Commit message: better net naming
Connections:
- net VCC renamed +5VDC
- net VDC renamed +6VDC
- net VEE renamed -5VDC
- net VPD_EN renamed 1V8_ENABLE
- net V_PD renamed 1V8DC
Other:
- sheet Channel0 ports: added +5VDC, -5VDC, 1V8DC; removed VCC, VEE, V_PD
- sheet Channel1 ports: added +5VDC, -5VDC, 1V8DC; removed VCC, VEE, V_PD
- sheet Channel2 ports: added +5VDC, -5VDC, 1V8DC; removed VCC, VEE, V_PD
- sheet Channel3 ports: added +5VDC, -5VDC, 1V8DC; removed VCC, VEE, V_PD
- note added: "This chip is essentially also a level shifter. The 'T' in SN74HCT stands for TTL - compatible. Its V_HIGH threshold is ~2V and V_LOW 0.8V, making it compatible for 3.3V input. The outputs are referenced to +5VDC, so 5V ish"
- note removed: "This chip is essentially also a level shifter. The 'T' in SN74HCT stands for TTL - compatible. Its V_HIGH threshold is ~2V and V_LOW 0.8V, making it compatible for 3.3V input. The outputs are referenced to VCC, so 5V ish"
Changed lines of the file:
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@@
 		)
 	)
-	(text "This chip is essentially also a level shifter. \nThe 'T' in SN74HCT stands for TTL - compatible.\nIts V_HIGH threshold is ~2V and V_LOW 0.8V, making \nit compatible for 3.3V input. The outputs are referenced\nto VCC, so 5V ish"
+	(text "This chip is essentially also a level shifter. \nThe 'T' in SN74HCT stands for TTL - compatible.\nIts V_HIGH threshold is ~2V and V_LOW 0.8V, making \nit compatible for 3.3V input. The outputs are referenced\nto +5VDC, so 5V ish"
 		(exclude_from_sim no)
 		(at 83.566 286.512 0)
@@
 	(wire
 		(pts
-			(xy 259.08 361.95) (xy 262.89 361.95)
+			(xy 261.62 361.95) (xy 262.89 361.95)
 		)
 		(stroke
@@
 		)
 	)
-	(global_label "VEE"
+	(global_label "-5VDC"
 		(shape input)
 		(at 139.7 373.38 180)
@@
 		)
 	)
-	(global_label "V_PD"
+	(global_label "1V8DC"
 		(shape input)
 		(at 167.64 477.52 0)
@@
 		)
 	)
-	(global_label "VDC"
+	(global_label "+6VDC"
 		(shape input)
 		(at 191.77 416.56 90)
@@
 		)
 	)
-	(global_label "VEE"
+	(global_label "-5VDC"
 		(shape input)
 		(at 77.47 469.9 180)
@@
 		)
 	)
-	(global_label "VDC"
+	(global_label "+6VDC"
 		(shape input)
 		(at 38.1 436.88 180)
@@
 		)
 	)
-	(global_label "V_PD"
+	(global_label "1V8DC"
 		(shape input)
 		(at 96.52 375.92 180)
@@
 		)
 	)
-	(global_label "VCC"
+	(global_label "+5VDC"
 		(shape input)
 		(at 166.37 457.2 180)
@@
 		)
 	)
-	(global_label "VEE"
+	(global_label "-5VDC"
 		(shape input)
 		(at 210.82 273.05 0)
@@
 		)
 	)
-	(global_label "VCC"
+	(global_label "+5VDC"
 		(shape input)
 		(at 139.7 370.84 180)
@@
 		)
 	)
-	(global_label "VEE"
+	(global_label "-5VDC"
 		(shape input)
 		(at 96.52 373.38 180)
@@
 		)
 	)
-	(global_label "VCC"
+	(global_label "+5VDC"
 		(shape input)
 		(at 53.34 370.84 180)
@@
 		)
 	)
-	(global_label "V_PD"
+	(global_label "1V8DC"
 		(shape input)
 		(at 182.88 375.92 180)
@@
 		)
 	)
-	(global_label "VCC"
+	(global_label "+5VDC"
 		(shape input)
 		(at 96.52 370.84 180)
@@
 		)
 	)
-	(global_label "VCC"
+	(global_label "+5VDC"
 		(shape input)
 		(at 417.83 344.17 0)
@@
 		)
 	)
-	(global_label "VCC"
+	(global_label "+5VDC"
 		(shape input)
 		(at 332.74 341.63 0)
@@
 		)
 	)
-	(global_label "VDC"
+	(global_label "+6VDC"
 		(shape input)
 		(at 77.47 402.59 0)
@@
 		)
 	)
-	(global_label "V_PD"
+	(global_label "1V8DC"
 		(shape input)
 		(at 53.34 375.92 180)
@@
 		)
 	)
-	(global_label "VCC"
+	(global_label "+5VDC"
 		(shape input)
 		(at 137.16 421.64 180)
@@
 		)
 	)
-	(global_label "VCC"
+	(global_label "+5VDC"
 		(shape input)
 		(at 114.3 474.98 180)
@@
 		)
 	)
-	(global_label "V_PD"
+	(global_label "1V8DC"
 		(shape input)
 		(at 210.82 283.21 0)
@@
 		)
 	)
-	(global_label "VCC"
+	(global_label "+5VDC"
 		(shape input)
 		(at 334.01 364.49 270)
@@
 		)
 	)
-	(global_label "VPD_EN"
+	(global_label "1V8_ENABLE"
 		(shape input)
-		(at 259.08 361.95 180)
+		(at 261.62 361.95 180)
 		(fields_autoplaced yes)
 		(effects
@@
 		)
 		(property "Intersheetrefs" "${INTERSHEET_REFS}"
-			(at 249.0191 361.95 0)
+			(at 251.5591 361.95 0)
 			(effects
 				(font
@@
 		)
 	)
-	(global_label "VPD_EN"
+	(global_label "1V8_ENABLE"
 		(shape input)
 		(at 124.46 480.06 180)
@@
 		)
 	)
-	(global_label "V_PD"
+	(global_label "1V8DC"
 		(shape input)
 		(at 139.7 375.92 180)
@@
 		)
 	)
-	(global_label "VCC"
+	(global_label "+5VDC"
 		(shape input)
 		(at 210.82 267.97 0)
@@
 		)
 	)
-	(global_label "VCC"
+	(global_label "+5VDC"
 		(shape input)
 		(at 158.75 252.73 0)
@@
 		)
 	)
-	(global_label "VEE"
+	(global_label "-5VDC"
 		(shape input)
 		(at 53.34 373.38 180)
@@
 		)
 	)
-	(global_label "VEE"
+	(global_label "-5VDC"
 		(shape input)
 		(at 182.88 373.38 180)
@@
 		)
 	)
-	(global_label "VCC"
+	(global_label "+5VDC"
 		(shape input)
 		(at 182.88 370.84 180)
@@
 			)
 		)
-		(pin "VCC" input
+		(pin "+5VDC" input
 			(at 96.52 370.84 180)
 			(effects
@@
 			)
 		)
-		(pin "VEE" input
+		(pin "-5VDC" input
 			(at 96.52 373.38 180)
 			(effects
@@
 			)
 		)
-		(pin "V_PD" input
+		(pin "1V8DC" input
 			(at 96.52 375.92 180)
 			(effects
@@
 			)
 		)
-		(pin "VCC" input
+		(pin "+5VDC" input
 			(at 53.34 370.84 180)
 			(effects
@@
 			)
 		)
-		(pin "VEE" input
+		(pin "-5VDC" input
 			(at 53.34 373.38 180)
 			(effects
@@
 			)
 		)
-		(pin "V_PD" input
+		(pin "1V8DC" input
 			(at 53.34 375.92 180)
 			(effects
@@
 			)
 		)
-		(pin "VCC" input
+		(pin "+5VDC" input
 			(at 139.7 370.84 180)
 			(effects
@@
 			)
 		)
-		(pin "VEE" input
+		(pin "-5VDC" input
 			(at 139.7 373.38 180)
 			(effects
@@
 			)
 		)
-		(pin "V_PD" input
+		(pin "1V8DC" input
 			(at 139.7 375.92 180)
 			(effects
@@
 			)
 		)
-		(pin "VCC" input
+		(pin "+5VDC" input
 			(at 182.88 370.84 180)
 			(effects
@@
 			)
 		)
-		(pin "VEE" input
+		(pin "-5VDC" input
 			(at 182.88 373.38 180)
 			(effects
@@
 			)
 		)
-		(pin "V_PD" input
+		(pin "1V8DC" input
 			(at 182.88 375.92 180)
 			(effects
