File: Hardware/STM32_EVAL/MiniMCU-STM32H573RIT6.kicad_pcb (KiCad board)
At the start: 4 copper layers, 47.8 x 35.1 mm, 48 parts, among them J1 TYPE-C-31-M-12, J10 DEBUG, J2 OUT, J3 Conn_01x12, J4 Conn_01x04, J5 Conn_01x08, J6 IN, J7 Conn_01x09, SW1 PTS810_SJM_250_SMTR_LFS, SW2 PTS810_SJM_250_SMTR_LFS, U1 USBLC6-2SC6, U2 LD1117S33TR, U3 SP3485CN-L, U4 STM32H573RIT6, Y1 ECS-80-18-23B-JTN-TR

Commit message: Updated STM32 Eval
Parts:
- moved R6 0.61 mm to (183.7, 92.3)
- moved D3 0.61 mm to (183.2, 91.2)
Changed lines of the file:
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@@
 	(footprint "MyParts:LTST-C190KGKT"
 		(layer "F.Cu")
-		(at 182.78 90.69)
+		(at 183.165 91.16)
 		(property "Reference" "D3"
-			(at 0 1 0)
+			(at 2.635 0.11 0)
 			(layer "F.SilkS")
 			(effects
@@
 	(footprint "Resistor_SMD:R_0402_1005Metric"
 		(layer "F.Cu")
-		(at 183.32 91.88 180)
+		(at 183.705 92.35 180)
 		(descr "Resistor SMD 0402 (1005 Metric), square (rectangular) end terminal, IPC_7351 nominal, (Body size source: IPC-SM-782 page 72, https://www.pcb-3d.com/wordpress/wp-content/uploads/ipc-sm-782a_amendment_1_and_2.pdf), generated with kicad-footprint-generator")
 		(tags "resistor")
 		(property "Reference" "R6"
-			(at 0 1 0)
+			(at -2.055 -0.23 0)
 			(layer "F.SilkS")
 			(effects
@@
 	)
 	(segment
+		(start 181.165 91.16)
+		(end 180.65 91.16)
+		(width 0.2)
+		(layer "F.Cu")
+		(net 1)
+	)
+	(segment
 		(start 190.4 111.2)
 		(end 190.5 111.3)
@@
 	)
 	(segment
-		(start 181.97 90.69)
-		(end 180.78 90.69)
+		(start 182.355 91.16)
+		(end 181.165 91.16)
 		(width 0.2)
 		(layer "F.Cu")
@@
 	)
 	(segment
-		(start 180.78 90.69)
-		(end 180.48 90.99)
-		(width 0.2)
-		(layer "F.Cu")
-		(net 1)
-	)
-	(segment
 		(start 197.45 117)
 		(end 197.45 116.25)
@@
 	)
 	(segment
+		(start 180.65 91.16)
+		(end 180.48 90.99)
+		(width 0.2)
+		(layer "F.Cu")
+		(net 1)
+	)
+	(segment
 		(start 204.9 120.36)
 		(end 204.9 120.5)
@@
 	)
 	(segment
-		(start 181.79 91.89)
-		(end 182.8 91.89)
+		(start 182.175 92.36)
+		(end 183.185 92.36)
 		(width 0.25)
 		(layer "F.Cu")
@@
 	)
 	(via
-		(at 181.79 91.89)
+		(at 182.175 92.36)
 		(size 0.6)
 		(drill 0.3)
@@
 	)
 	(segment
-		(start 183.81 91.85)
-		(end 183.81 90.91)
+		(start 184.195 92.32)
+		(end 184.195 91.38)
 		(width 0.25)
 		(layer "F.Cu")
